File: KiCad/Examples/impeller18/can.kicad_sch (KiCad schematic)
At the start: 64 parts, among them J10 PLS-5, J11 430450400, J12 PLS-3, J13 PLS-5, J14 430450400, J15 PLS-3, SW8 MSS-12D16, SW9 MSS-12D16, U10 ISO1050DUB, U11 ISO1050DUB, U12 MCP2515-I/SO, U13 B0505MT-1WR4, U14 ISO1050DUB, U15 ISO1050DUB, U16 MCP2515-I/SO, U17 B0505MT-1WR4, Y3 X322516MLB4SI, Y4 X322516MLB4SI

Commit message: 23.03.2025
Changed lines of the file:
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@@
 (kicad_sch
-	(version 20231120)
+	(version 20250114)
 	(generator "eeschema")
-	(generator_version "8.0")
+	(generator_version "9.0")
 	(paper "A3")
+	(rectangle
+		(start 26.035 125.095)
+		(end 322.58 219.71)
+		(stroke
+			(width 0)
+			(type default)
+		)
+		(fill
+			(type none)
+		)
+	)
+	(rectangle
+		(start 26.035 24.765)
+		(end 322.58 119.38)
+		(stroke
+			(width 0)
+			(type default)
+		)
+		(fill
+			(type none)
+		)
+	)
+	(text "https://files.waveshare.com/upload/1/15/2-CH-CAN-HAT-Schematic.pdf\nшилд"
+		(exclude_from_sim no)
+		(at 275.59 213.995 0)
+		(effects
+			(font
+				(size 1.27 1.27)
+			)
+		)
+	)
+	(text "https://files.waveshare.com/upload/1/15/2-CH-CAN-HAT-Schematic.pdf\nшилд"
+		(exclude_from_sim no)
+		(at 275.59 113.665 0)
+		(effects
+			(font
+				(size 1.27 1.27)
+			)
+		)
+	)
+	(text "+gnd"
+		(exclude_from_sim no)
+		(at 264.795 204.47 0)
+		(effects
+			(font
+				(size 5 5)
+			)
+		)
+	)
 	(junction
 		(at 253.365 82.55)
@@
 		)
 	)
-	(rectangle
-		(start 26.035 125.095)
-		(end 322.58 219.71)
-		(stroke
-			(width 0)
-			(type default)
-		)
-		(fill
-			(type none)
-		)
-	)
-	(rectangle
-		(start 26.035 24.765)
-		(end 322.58 119.38)
-		(stroke
-			(width 0)
-			(type default)
-		)
-		(fill
-			(type none)
-		)
-	)
-	(text "https://files.waveshare.com/upload/1/15/2-CH-CAN-HAT-Schematic.pdf\nшилд"
-		(exclude_from_sim no)
-		(at 275.59 213.995 0)
-		(effects
-			(font
-				(size 1.27 1.27)
-			)
-		)
-	)
-	(text "https://files.waveshare.com/upload/1/15/2-CH-CAN-HAT-Schematic.pdf\nшилд"
-		(exclude_from_sim no)
-		(at 275.59 113.665 0)
-		(effects
-			(font
-				(size 1.27 1.27)
-			)
-		)
-	)
-	(text "+gnd"
-		(exclude_from_sim no)
-		(at 264.795 204.47 0)
-		(effects
-			(font
-				(size 5 5)
-			)
-		)
-	)
 	(label "CAN1_RPi_TX"
 		(at 201.295 172.72 180)
-		(fields_autoplaced yes)
 		(effects
 			(font
@@
 	(label "CAN0_RPi_RX"
 		(at 250.19 38.735 0)
-		(fields_autoplaced yes)
 		(effects
 			(font
@@
 	(label "CAN1_-"
 		(at 157.48 170.18 0)
-		(fields_autoplaced yes)
 		(effects
 			(font
@@
 	(label "CAN1_RPi_RX"
 		(at 315.595 165.1 180)
-		(fields_autoplaced yes)
 		(effects
 			(font
@@
 	(label "CAN0+"
 		(at 74.295 50.8 180)
-		(fields_autoplaced yes)
 		(effects
 			(font
@@
 	(label "CAN1_-"
 		(at 157.48 141.605 0)
-		(fields_autoplaced yes)
 		(effects
 			(font
@@
 	(label "CAN0_RPi_TX"
 		(at 201.295 72.39 180)
-		(fields_autoplaced yes)
 		(effects
 			(font
@@
 	(label "CAN1+"
 		(at 74.295 151.13 180)
-		(fields_autoplaced yes)
 		(effects
 			(font
@@
 	(label "CAN0_RPi_TX"
 		(at 250.19 41.275 0)
-		(fields_autoplaced yes)
 		(effects
 			(font
@@
 	(label "CAN0_+"
 		(at 157.48 72.39 0)
-		(fields_autoplaced yes)
 		(effects
 			(font
@@
 	(label "CAN0_-"
 		(at 113.665 45.72 180)
-		(fields_autoplaced yes)
 		(effects
 			(font
@@
 	(label "CAN0_RPi_RX"
 		(at 201.295 69.85 180)
-		(fields_autoplaced yes)
 		(effects
 			(font
@@
 	(label "CAN1_RPi_RX"
 		(at 254 139.7 0)
-		(fields_autoplaced yes)
 		(effects
 			(font
@@
 	(label "CAN0_-"
 		(at 157.48 41.275 0)
-		(fields_autoplaced yes)
 		(effects
 			(font
@@
 	(label "CAN1_RPi_RX"
 		(at 201.295 170.18 180)
-		(fields_autoplaced yes)
 		(effects
 			(font
@@
 	(label "CAN0_RPi_TX"
 		(at 315.595 67.31 180)
-		(fields_autoplaced yes)
 		(effects
 			(font
@@
 	(label "CAN1_RPi_TX"
 		(at 254 142.24 0)
-		(fields_autoplaced yes)
 		(effects
 			(font
@@
 	(label "CAN0-"
 		(at 74.295 45.72 180)
-		(fields_autoplaced yes)
 		(effects
 			(font
@@
 	(label "CAN1_+"
 		(at 114.3 151.13 180)
-		(fields_autoplaced yes)
 		(effects
 			(font
@@
 	(label "CAN1_+"
 		(at 157.48 172.72 0)
-		(fields_autoplaced yes)
 		(effects
 			(font
@@
 	(label "CAN0_RPi_RX"
 		(at 315.595 64.77 180)
-		(fields_autoplaced yes)
 		(effects
 			(font
@@
 	(label "CAN1_+"
 		(at 157.48 144.145 0)
-		(fields_autoplaced yes)
 		(effects
 			(font
@@
 	(label "CAN1-"
 		(at 74.295 146.05 180)
-		(fields_autoplaced yes)
 		(effects
 			(font
@@
 	(label "CAN0_+"
 		(at 157.48 43.815 0)
-		(fields_autoplaced yes)
 		(effects
 			(font
@@
 	(label "CAN0_-"
 		(at 157.48 69.85 0)
-		(fields_autoplaced yes)
 		(effects
 			(font
@@
 	(label "CAN0_+"
 		(at 113.665 50.8 180)
-		(fields_autoplaced yes)
 		(effects
 			(font
@@
 	(label "CAN1_-"
 		(at 114.3 146.05 180)
-		(fields_autoplaced yes)
 		(effects
 			(font
@@
 	(label "CAN1_RPi_TX"
 		(at 315.595 167.64 180)
-		(fields_autoplaced yes)
 		(effects
 			(font
