File: KiCad/Examples/impeller18/power.kicad_sch (KiCad schematic)
At the start: 123 parts, among them J6 430450400, J7 PLS-2, J8 PLS-2, J9 PLS-2, K1 1393219-3, K2 1393219-3, K3 1393219-3, Q1 BSS138, Q2 AO3401A, Q3 BSS138, Q4 BSS138, Q5 BSS138, U2 LDL1117S33R, U3 VDRI25W05, U4 VDRI15W12, U5 HY2213-BB3A, U6 bq2057WSN, U7 HY2213-BB3A, U8 LD1084V, U9 MCP3001-I/SN

Commit message: 23.03.2025
Changed lines of the file:
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@@
 (kicad_sch
-	(version 20231120)
+	(version 20250114)
 	(generator "eeschema")
-	(generator_version "8.0")
+	(generator_version "9.0")
 	(paper "A3")
+	(text "390-5.31\n400-5.4"
+		(exclude_from_sim no)
+		(at 353.695 245.745 0)
+		(effects
+			(font
+				(size 1.27 1.27)
+			)
+		)
+	)
 	(junction
 		(at 91.44 83.82)
@@
 		)
 	)
-	(text "390-5.31\n400-5.4"
-		(exclude_from_sim no)
-		(at 353.695 245.745 0)
-		(effects
-			(font
-				(size 1.27 1.27)
-			)
-		)
-	)
 	(label "BAT_RELAY_TOGGLE_"
 		(at 283.845 149.86 180)
-		(fields_autoplaced yes)
 		(effects
 			(font
@@
 	(label "BAT_CHRG_TOGGLE_"
 		(at 325.755 121.285 0)
-		(fields_autoplaced yes)
 		(effects
 			(font
@@
 	(label "BAT_CHRG_TOGGLE_"
 		(at 240.03 152.4 180)
-		(fields_autoplaced yes)
 		(effects
 			(font
@@
 	(label "BAT_CHRG_TOGGLE_"
 		(at 240.03 186.055 180)
-		(fields_autoplaced yes)
 		(effects
 			(font
@@
 	(label "BAT_RELAY_TOGGLE_"
 		(at 325.755 149.225 0)
-		(fields_autoplaced yes)
 		(effects
 			(font
