File: KiCad/BMS/can.kicad_sch (KiCad schematic)
At the start: 9 parts, among them J3 430450400, J5 Conn_01x03, U2 ISO1050DUB

Commit message: 14.03.2025
Parts:
- renumbered J5 to J4
Changed lines of the file:
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@@
 		(on_board yes)
 		(dnp no)
-		(property "Reference" "J5"
+		(property "Reference" "J4"
 			(at 180.848 81.788 0)
 			(effects
@@
 			(project "BMS"
 				(path "/d2402062-308b-4eb4-ada9-28eaf3edc216/b4d93d65-8b92-4fd1-a768-223386b4c558"
-					(reference "J5")
+					(reference "J4")
 					(unit 1)
 				)

Commit message: 22.03.2025
Parts:
- added C25: C_Small, symbol Device:C_Small
Connections:
- net CAN0+: now also D1.2 (K); no longer D1.1 (K)
- net CAN0-: now also D1.1 (K); no longer D1.2 (K)
Other:
- moved on the sheet: L1

Commit message: 23.03.2025
Parts:
- removed C25: C_Small, symbol Device:C_Small
Other:
- note removed: "CAN Connector"
- note removed: "EMC"
- note removed: "ESD PROTECT"
- note removed: "ISO1050DUB"
- note removed: "Terminator"
- moved on the sheet: C13, C14, C15, D1, J3, J4, L1, R3, U2
