File: KiCad/BMS/can.kicad_sch (KiCad schematic)
At the start: 12 parts, among them J3 430450400, J4 Conn_01x03, U2 ISO1050DUB, U3 B0505MT

Commit message: 08.04.2025
Parts:
- renumbered R3 to R2
Changed lines of the file:
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@@
 		(dnp no)
 		(fields_autoplaced yes)
-		(property "Reference" "#PWR079"
+		(property "Reference" "#PWR015"
 			(at 178.435 46.99 0)
 			(effects
@@
 			(project "BMS"
 				(path "/d2402062-308b-4eb4-ada9-28eaf3edc216/b4d93d65-8b92-4fd1-a768-223386b4c558"
-					(reference "#PWR079")
+					(reference "#PWR015")
 					(unit 1)
 				)
@@
 		(dnp no)
 		(fields_autoplaced yes)
-		(property "Reference" "#PWR029"
+		(property "Reference" "#PWR028"
 			(at 132.715 106.68 0)
 			(effects
@@
 			(project "BMS"
 				(path "/d2402062-308b-4eb4-ada9-28eaf3edc216/b4d93d65-8b92-4fd1-a768-223386b4c558"
-					(reference "#PWR029")
+					(reference "#PWR028")
 					(unit 1)
 				)
@@
 		(on_board yes)
 		(dnp no)
-		(property "Reference" "#PWR027"
+		(property "Reference" "#PWR026"
 			(at 117.475 100.33 0)
 			(effects
@@
 			(project "BMS"
 				(path "/d2402062-308b-4eb4-ada9-28eaf3edc216/b4d93d65-8b92-4fd1-a768-223386b4c558"
-					(reference "#PWR027")
+					(reference "#PWR026")
 					(unit 1)
 				)
@@
 		(dnp no)
 		(fields_autoplaced yes)
-		(property "Reference" "#PWR025"
+		(property "Reference" "#PWR024"
 			(at 209.55 95.25 0)
 			(effects
@@
 			(project "BMS"
 				(path "/d2402062-308b-4eb4-ada9-28eaf3edc216/b4d93d65-8b92-4fd1-a768-223386b4c558"
-					(reference "#PWR025")
+					(reference "#PWR024")
 					(unit 1)
 				)
@@
 		(dnp no)
 		(fields_autoplaced yes)
-		(property "Reference" "#PWR022"
+		(property "Reference" "#PWR021"
 			(at 106.045 83.82 0)
 			(effects
@@
 			(project "BMS"
 				(path "/d2402062-308b-4eb4-ada9-28eaf3edc216/b4d93d65-8b92-4fd1-a768-223386b4c558"
-					(reference "#PWR022")
+					(reference "#PWR021")
 					(unit 1)
 				)
@@
 		(dnp no)
 		(fields_autoplaced yes)
-		(property "Reference" "#PWR018"
+		(property "Reference" "#PWR017"
 			(at 178.435 68.58 0)
 			(effects
@@
 			(project "BMS"
 				(path "/d2402062-308b-4eb4-ada9-28eaf3edc216/b4d93d65-8b92-4fd1-a768-223386b4c558"
-					(reference "#PWR018")
+					(reference "#PWR017")
 					(unit 1)
 				)
@@
 		(on_board yes)
 		(dnp no)
-		(property "Reference" "#PWR028"
+		(property "Reference" "#PWR027"
 			(at 142.875 105.41 0)
 			(effects
@@
 			(project "BMS"
 				(path "/d2402062-308b-4eb4-ada9-28eaf3edc216/b4d93d65-8b92-4fd1-a768-223386b4c558"
-					(reference "#PWR028")
+					(reference "#PWR027")
 					(unit 1)
 				)
@@
 		(dnp no)
 		(fields_autoplaced yes)
-		(property "Reference" "#PWR024"
+		(property "Reference" "#PWR023"
 			(at 167.64 95.25 0)
 			(effects
@@
 			(project "BMS"
 				(path "/d2402062-308b-4eb4-ada9-28eaf3edc216/b4d93d65-8b92-4fd1-a768-223386b4c558"
-					(reference "#PWR024")
+					(reference "#PWR023")
 					(unit 1)
 				)
@@
 		(dnp no)
 		(fields_autoplaced yes)
-		(property "Reference" "#PWR021"
+		(property "Reference" "#PWR019"
 			(at 132.715 76.2 0)
 			(effects
@@
 			(project "BMS"
 				(path "/d2402062-308b-4eb4-ada9-28eaf3edc216/b4d93d65-8b92-4fd1-a768-223386b4c558"
-					(reference "#PWR021")
+					(reference "#PWR019")
 					(unit 1)
 				)
@@
 		(on_board yes)
 		(dnp no)
-		(property "Reference" "#PWR023"
+		(property "Reference" "#PWR022"
 			(at 117.475 83.82 0)
 			(effects
@@
 			(project "BMS"
 				(path "/d2402062-308b-4eb4-ada9-28eaf3edc216/b4d93d65-8b92-4fd1-a768-223386b4c558"
-					(reference "#PWR023")
+					(reference "#PWR022")
 					(unit 1)
 				)
@@
 		(on_board yes)
 		(dnp no)
-		(property "Reference" "R3"
+		(property "Reference" "R2"
 			(at 258.445 77.978 90)
 			(effects
@@
 			(project "BMS"
 				(path "/d2402062-308b-4eb4-ada9-28eaf3edc216/b4d93d65-8b92-4fd1-a768-223386b4c558"
-					(reference "R3")
+					(reference "R2")
 					(unit 1)
 				)
@@
 		(dnp no)
 		(fields_autoplaced yes)
-		(property "Reference" "#PWR026"
+		(property "Reference" "#PWR025"
 			(at 106.045 100.33 0)
 			(effects
@@
 			(project "BMS"
 				(path "/d2402062-308b-4eb4-ada9-28eaf3edc216/b4d93d65-8b92-4fd1-a768-223386b4c558"
-					(reference "#PWR026")
+					(reference "#PWR025")
 					(unit 1)
 				)
@@
 		(dnp no)
 		(fields_autoplaced yes)
-		(property "Reference" "#PWR017"
+		(property "Reference" "#PWR016"
 			(at 257.175 48.26 0)
 			(effects
@@
 			(project "BMS"
 				(path "/d2402062-308b-4eb4-ada9-28eaf3edc216/b4d93d65-8b92-4fd1-a768-223386b4c558"
-					(reference "#PWR017")
+					(reference "#PWR016")
 					(unit 1)
 				)
@@
 		(dnp no)
 		(fields_autoplaced yes)
-		(property "Reference" "#PWR019"
+		(property "Reference" "#PWR018"
 			(at 257.175 68.58 0)
 			(effects
@@
 			(project "BMS"
 				(path "/d2402062-308b-4eb4-ada9-28eaf3edc216/b4d93d65-8b92-4fd1-a768-223386b4c558"
-					(reference "#PWR019")
-					(unit 1)
-				)
+					(reference "#PWR018")
+					(unit 1)
+				)

Commit message: pupupu
Connections:
- net 3v3 renamed 3V3
Changed lines of the file:
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@@
 			)
 		)
-		(property "Value" "3v3"
-			(at 257.175 39.37 0)
+		(property "Value" "3V3"
+			(at 259.08 43.1799 0)
 			(effects
 				(font
 					(size 1.27 1.27)
 				)
+				(justify left)
 			)
 		)

Commit message: 19.04.2025
Parts:
- renumbered R2 to R3
Connections:
- net GND_CAN: no longer J3.2 (Pin_2)
- no-connect marks 1 -> 2
Other:
- moved on the sheet: L1
