File: KiCad/BMS/BMS.kicad_pcb (KiCad board)
At the start: 4 copper layers, 413.4 x 187.5 mm, 199 parts, among them J1 PLS-6, J2 BH1,27-10-G, J3 430450400, J4 430451200, J5 Conn_01x03, Q1 PNP, Q10 NMOS, Q11 PNP, Q12 BSS138, Q13 NMOS, Q14 PNP, Q15 NMOS, Q16 PNP, Q17 NMOS, Q2 NMOS, Q3 PNP, Q4 NMOS, Q5 PNP, Q6 NMOS, Q7 PNP, Q8 NMOS, Q9 PNP, SW1 B3F1060, SW2 MSS-12D16, U1 STM32F405RGTx, U10 TL431, U11 B0505MT, U12 MCP3201, U13 TL431, U14 HCPL-0630, U15 TL431, U16 HCPL-0600, U17 TL431, U18 HCPL-0600, U19 TL431, U2 ISO1050DUB, U20 TL431, U21 74HC4051, U22 MCP3201, U23 HCPL-0630, U3 ST1S14PHR, U4 LDL1117S33R, U5 HCPL-0630, U6 TL431, U7 74HC4051, U8 HCPL-0630, U9 TL431, Y1 Crystal

Commit message: 12_03_2025 update
Parts:
- moved C18 38.9 mm to (405.5, -102.1), turned to -90 degrees
- moved C19 34.4 mm to (404.0, -102.1), turned to -90 degrees
- moved C17 31.5 mm to (440.8, -76.2)
- moved L2 31.5 mm to (431.8, -77.2)
- moved D12 5.93 mm to (215.1, -22.5)
- moved Q8 0.79 mm to (96.7, -48.0)
Routing:
- net Net-(U13-K): track 23.3 -> 0.00 mm
- net 24V0: track 0.00 -> 11.5 mm, vias 0 -> 1
- net GND: track 15.9 -> 18.4 mm, vias 5 -> 6
Changed lines of the file:
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@@
 	(footprint "Capacitor_SMD:C_0603_1608Metric"
 		(layer "F.Cu")
-		(at 367 -108)
+		(at 405.49 -102.085 -90)
 		(descr "Capacitor SMD 0603 (1608 Metric), square (rectangular) end terminal, IPC_7351 nominal, (Body size source: IPC-SM-782 page 76, https://www.pcb-3d.com/wordpress/wp-content/uploads/ipc-sm-782a_amendment_1_and_2.pdf), generated with kicad-footprint-generator")
 		(tags "capacitor")
 		(property "Reference" "C18"
-			(at 0 -1.43 0)
+			(at 0 -1.43 90)
 			(layer "F.SilkS")
 			(effects
@@
 		)
 		(property "Value" "10u"
-			(at 0 1.5 0)
+			(at 0 1.5 90)
 			(layer "F.Fab")
 			(effects
@@
 		)
 		(property "Datasheet" ""
-			(at 0 0 0)
+			(at 0 0 270)
 			(unlocked yes)
 			(layer "F.Fab")
@@
 		)
 		(property "Description" "Unpolarized capacitor"
-			(at 0 0 0)
+			(at 0 0 270)
 			(unlocked yes)
 			(layer "F.Fab")
@@
 		(attr smd)
 		(fp_line
-			(start -0.14058 -0.51)
-			(end 0.14058 -0.51)
+			(start -0.14058 0.51)
+			(end 0.14058 0.51)
 			(stroke
 				(width 0.12)
@@
 		)
 		(fp_line
-			(start -0.14058 0.51)
-			(end 0.14058 0.51)
+			(start -0.14058 -0.51)
+			(end 0.14058 -0.51)
 			(stroke
 				(width 0.12)
@@
 		)
 		(fp_line
-			(start -1.48 -0.73)
-			(end 1.48 -0.73)
+			(start -1.48 0.73)
+			(end -1.48 -0.73)
 			(stroke
 				(width 0.05)
@@
 		)
 		(fp_line
-			(start -1.48 0.73)
-			(end -1.48 -0.73)
+			(start 1.48 0.73)
+			(end -1.48 0.73)
 			(stroke
 				(width 0.05)
@@
 		)
 		(fp_line
-			(start 1.48 -0.73)
-			(end 1.48 0.73)
+			(start -1.48 -0.73)
+			(end 1.48 -0.73)
 			(stroke
 				(width 0.05)
@@
 		)
 		(fp_line
-			(start 1.48 0.73)
-			(end -1.48 0.73)
+			(start 1.48 -0.73)
+			(end 1.48 0.73)
 			(stroke
 				(width 0.05)
@@
 		)
 		(fp_line
-			(start -0.8 -0.4)
-			(end 0.8 -0.4)
+			(start -0.8 0.4)
+			(end -0.8 -0.4)
 			(stroke
 				(width 0.1)
@@
 		)
 		(fp_line
-			(start -0.8 0.4)
-			(end -0.8 -0.4)
+			(start 0.8 0.4)
+			(end -0.8 0.4)
 			(stroke
 				(width 0.1)
@@
 		)
 		(fp_line
-			(start 0.8 -0.4)
-			(end 0.8 0.4)
+			(start -0.8 -0.4)
+			(end 0.8 -0.4)
 			(stroke
 				(width 0.1)
@@
 		)
 		(fp_line
-			(start 0.8 0.4)
-			(end -0.8 0.4)
+			(start 0.8 -0.4)
+			(end 0.8 0.4)
 			(stroke
 				(width 0.1)
@@
 		)
 		(fp_text user "${REFERENCE}"
-			(at 0 0 0)
+			(at 0 0 90)
 			(layer "F.Fab")
 			(effects
@@
 		)
 		(pad "1" smd roundrect
-			(at -0.775 0)
+			(at -0.775 0 270)
 			(size 0.9 0.95)
 			(layers "F.Cu" "F.Mask" "F.Paste")
@@
 		)
 		(pad "2" smd roundrect
-			(at 0.775 0)
+			(at 0.775 0 270)
 			(size 0.9 0.95)
 			(layers "F.Cu" "F.Mask" "F.Paste")
@@
 	(footprint "user:CTSFW7050F"
 		(layer "F.Cu")
-		(at 405.5 -94.5 180)
+		(at 431.8 -77.24 180)
 		(property "Reference" "L2"
 			(at 0 -4.5 180)
@@
 	(footprint "Package_TO_SOT_SMD:TO-252-2"
 		(layer "F.Cu")
-		(at 97.423 -47.603)
+		(at 96.74 -48)
 		(descr "TO-252/DPAK SMD package, http://www.infineon.com/cms/en/product/packages/PG-TO252/PG-TO252-3-1/")
 		(tags "DPAK TO-252 DPAK-3 TO-252-3 SOT-428")
@@
 	(footprint "Capacitor_SMD:C_0603_1608Metric"
 		(layer "F.Cu")
-		(at 369.725 -99.5)
+		(at 404.03 -102.085 -90)
 		(descr "Capacitor SMD 0603 (1608 Metric), square (rectangular) end terminal, IPC_7351 nominal, (Body size source: IPC-SM-782 page 76, https://www.pcb-3d.com/wordpress/wp-content/uploads/ipc-sm-782a_amendment_1_and_2.pdf), generated with kicad-footprint-generator")
 		(tags "capacitor")
 		(property "Reference" "C19"
-			(at 0 -1.43 0)
+			(at 0 -1.43 90)
 			(layer "F.SilkS")
 			(effects
@@
 		)
 		(property "Value" "100n"
-			(at 0 1.43 0)
+			(at 0 1.43 90)
 			(layer "F.Fab")
 			(effects
@@
 		)
 		(property "Datasheet" ""
-			(at 0 0 0)
+			(at 0 0 270)
 			(unlocked yes)
 			(layer "F.Fab")
@@
 		)
 		(property "Description" "Unpolarized capacitor"
-			(at 0 0 0)
+			(at 0 0 270)
 			(unlocked yes)
 			(layer "F.Fab")
@@
 		(attr smd)
 		(fp_line
-			(start -0.14058 -0.51)
-			(end 0.14058 -0.51)
+			(start -0.14058 0.51)
+			(end 0.14058 0.51)
 			(stroke
 				(width 0.12)
@@
 		)
 		(fp_line
-			(start -0.14058 0.51)
-			(end 0.14058 0.51)
+			(start -0.14058 -0.51)
+			(end 0.14058 -0.51)
 			(stroke
 				(width 0.12)
@@
 		)
 		(fp_line
-			(start -1.48 -0.73)
-			(end 1.48 -0.73)
+			(start -1.48 0.73)
+			(end -1.48 -0.73)
 			(stroke
 				(width 0.05)
@@
 		)
 		(fp_line
-			(start -1.48 0.73)
-			(end -1.48 -0.73)
+			(start 1.48 0.73)
+			(end -1.48 0.73)
 			(stroke
 				(width 0.05)
@@
 		)
 		(fp_line
-			(start 1.48 -0.73)
-			(end 1.48 0.73)
+			(start -1.48 -0.73)
+			(end 1.48 -0.73)
 			(stroke
 				(width 0.05)
@@
 		)
 		(fp_line
-			(start 1.48 0.73)
-			(end -1.48 0.73)
+			(start 1.48 -0.73)
+			(end 1.48 0.73)
 			(stroke
 				(width 0.05)
@@
 		)
 		(fp_line
-			(start -0.8 -0.4)
-			(end 0.8 -0.4)
+			(start -0.8 0.4)
+			(end -0.8 -0.4)
 			(stroke
 				(width 0.1)
@@
 		)
 		(fp_line
-			(start -0.8 0.4)
-			(end -0.8 -0.4)
+			(start 0.8 0.4)
+			(end -0.8 0.4)
 			(stroke
 				(width 0.1)
@@
 		)
 		(fp_line
-			(start 0.8 -0.4)
-			(end 0.8 0.4)
+			(start -0.8 -0.4)
+			(end 0.8 -0.4)
 			(stroke
 				(width 0.1)
@@
 		)
 		(fp_line
-			(start 0.8 0.4)
-			(end -0.8 0.4)
+			(start 0.8 -0.4)
+			(end 0.8 0.4)
 			(stroke
 				(width 0.1)
@@
 		)
 		(fp_text user "${REFERENCE}"
-			(at 0 0 0)
+			(at 0 0 90)
 			(layer "F.Fab")
 			(effects
@@
 		)
 		(pad "1" smd roundrect
-			(at -0.775 0)
+			(at -0.775 0 270)
 			(size 0.9 0.95)
 			(layers "F.Cu" "F.Mask" "F.Paste")
@@
 		)
 		(pad "2" smd roundrect
-			(at 0.775 0)
+			(at 0.775 0 270)
 			(size 0.9 0.95)
 			(layers "F.Cu" "F.Mask" "F.Paste")
@@
 	(footprint "Capacitor_THT:CP_Radial_D5.0mm_P2.00mm"
 		(layer "F.Cu")
-		(at 414.5 -93.5 -90)
+		(at 440.8 -76.24 -90)
 		(descr "CP, Radial series, Radial, pin pitch=2.00mm, , diameter=5mm, Electrolytic Capacitor")
 		(tags "CP Radial series Radial pin pitch 2.00mm  diameter 5mm Electrolytic Capacitor")
@@
 	(footprint "LED_SMD:LED_1206_3216Metric"
 		(layer "F.Cu")
-		(at 209.175 -22.56)
+		(at 215.1 -22.5)
 		(descr "LED SMD 1206 (3216 Metric), square (rectangular) end terminal, IPC_7351 nominal, (Body size source: http://www.tortai-tech.com/upload/download/2011102023233369053.pdf), generated with kicad-footprint-generator")
 		(tags "LED")
@@
 	)
 	(segment
+		(start 404.03 -101.31)
+		(end 405.49 -101.31)
+		(width 0.9)
+		(layer "F.Cu")
+		(net 1)
+	)
+	(segment
 		(start 124.327 90.957)
 		(end 124.327 90.908)
@@
 	)
 	(segment
+		(start 405.49 -101.31)
+		(end 406.6 -101.31)
+		(width 0.6)
+		(layer "F.Cu")
+		(net 1)
+	)
+	(segment
 		(start 134.414 94.1)
 		(end 135.521 94.1)
@@
 	)
 	(via
+		(at 406.6 -101.31)
+		(size 0.6)
+		(drill 0.3)
+		(layers "F.Cu" "B.Cu")
+		(net 1)
+	)
+	(via
 		(at 116.635 101.324)
 		(size 0.6)
@@
 	)
 	(segment
-		(start 121.309 98.15)
-		(end 119.5 98.15)
-		(width 0.3)
+		(start 402.63 -100.62)
+		(end 402.33 -100.32)
+		(width 0.6)
 		(layer "F.Cu")
-		(net 49)
+		(net 14)
 	)
 	(segment
-		(start 86.7 -47.456)
-		(end 85.724 -46.48)
+		(start 401.97 -102.86)
+		(end 402.63 -102.2)
 		(width 0.6)
 		(layer "F.Cu")
-		(net 83)
+		(net 14)
 	)
 	(segment
-		(start 104.559 -46.899)
-		(end 102.79 -48.668)
+		(start 400.1775 -102.86)
+		(end 401.97 -102.86)
 		(width 0.6)
 		(layer "F.Cu")
-		(net 83)
+		(net 14)
 	)
 	(segment
-		(start 101.951002 -51.004)
-		(end 90.899 -51.004)
-		(width 0.6)
+		(start 404.03 -102.86)
+		(end 405.49 -102.86)
+		(width 0.9)
 		(layer "F.Cu")
-		(net 83)
+		(net 14)
 	)
 	(segment
-		(start 87.351 -47.456)
-		(end 86.7 -47.456)
+		(start 402.33 -100.32)
+		(end 400.1775 -100.32)
 		(width 0.6)
 		(layer "F.Cu")
-		(net 83)
+		(net 14)
 	)
 	(segment
-		(start 90.899 -51.004)
-		(end 87.351 -47.456)
+		(start 401.97 -102.86)
+		(end 404.03 -102.86)
 		(width 0.6)
 		(layer "F.Cu")
-		(net 83)
+		(net 14)
 	)
 	(segment
-		(start 102.79 -50.165004)
-		(end 101.951002 -51.004)
+		(start 405.49 -102.86)
+		(end 406.6 -102.86)
 		(width 0.6)
 		(layer "F.Cu")
-		(net 83)
+		(net 14)
 	)
 	(segment
-		(start 102.79 -48.668)
-		(end 102.79 -50.165004)
+		(start 402.63 -102.2)
+		(end 402.63 -100.62)
 		(width 0.6)
 		(layer "F.Cu")
-		(net 83)
+		(net 14)
+	)
+	(via
+		(at 406.6 -102.86)
+		(size 0.6)
+		(drill 0.3)
+		(layers "F.Cu" "B.Cu")
+		(net 14)
+	)
+	(segment
+		(start 121.309 98.15)
+		(end 119.5 98.15)
+		(width 0.3)
+		(layer "F.Cu")
+		(net 49)
 	)
 	(zone

Commit message: 14.03.2025
Parts:
- removed D10, D11, D12, D3, D4, D5, D8, D9: LED_B, LED_SMD:LED_1206_3216Metric
- removed R19, R30, R50, R74, R8, R85: 180, Resistor_SMD:R_0603_1608Metric
- removed the R41 at (86.5, -51.5)
- removed the R64 at (-128.2, -22.9)
- removed the U6 at (-113.9, -21.8)
- removed the U9 at (-113.9, -8.61)
- added U5: TL432DBZ, Package_TO_SOT_SMD:SOT-23, B.Cu at (185.6, 78.8)
- added U8: TL432DBZ, Package_TO_SOT_SMD:SOT-23, B.Cu at (175.5, 78.8)
- Q1, Q11, Q14, Q16, Q3, Q5, Q7, Q9, R16, R18, R21, R22, R29, R32, R33, R43, R44, R47, R49, R58, R60, R66, R67, R7, R71, R73, R77, R78, R82, R84, R86, R87, R89: moved to B.Cu
- R10: renamed from R11; moved to B.Cu
- R11: renamed from R12; moved to B.Cu
- R26: renamed from R27; moved to B.Cu
- R36: renamed from R37; moved to B.Cu
- R39: renamed from R40; moved to B.Cu
- R4: value 10k -> 47k
- R5: value 10k -> 4k7
- R53: renamed from R54; moved to B.Cu
- R54: renamed from R55; moved to B.Cu
- R6: value 10k -> 2k7
- R_bal_1, R_bal_2, R_bal_3, R_bal_4, R_bal_5, R_bal_6, R_bal_7, R_bal_8: footprint Resistor_SMD:R_0603_1608Metric -> Resistor_SMD:R_1206_3216Metric; moved to B.Cu
- U10, U13, U15, U17, U19, U20: value TL431 -> TL432DBZ; footprint Package_SO:SOIC-8_3.9x4.9mm_P1.27mm -> Package_TO_SOT_SMD:SOT-23; moved to B.Cu
- moved C17 441.1 mm to (51.7, 131.5)
- moved L2 441.1 mm to (42.7, 130.5)
- moved C22 414.9 mm to (28.9, 121.9)
- moved R6 414.9 mm to (21.3, 126.9)
- moved C16 414.9 mm to (19.8, 111.4)
- moved C18 414.9 mm to (52.1, 115.3)
- moved C19 414.9 mm to (50.7, 115.3)
- moved D2 414.9 mm to (41.6, 124.0)
- moved R4 414.9 mm to (29.1, 127.9)
- moved R5 414.9 mm to (32.5, 132.4)
- moved U3 414.9 mm to (44.0, 115.2)
- moved Q1 369.7 mm to (185.8, 82.8), turned to -90 degrees
- moved Q2 362.7 mm to (187.3, 79.2), turned to -90 degrees
- moved Q3 358.7 mm to (175.7, 82.8), turned to -90 degrees
- moved Q4 350.8 mm to (177.1, 79.2), turned to -90 degrees
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- renumbered C9 to C10, C10 to C9, J5 to J4, J4 to J5, R14 to R12, R15 to R13, R10 to R14, R13 to R15, R24 to R23, R25 to R24, R23 to R25, R28 to R27, R26 to R28, R38 to R37, R36 to R38, R39 to R41, R52 to R51, R51 to R52, R53 to R55, R57 to R56, R56 to R57, R61 to R62, R62 to R63, R63 to R64, R69 to R68, R70 to R69, R68 to R70, U5 to U6, U8 to U9
Connections:
- U10 pad 1: Net-(U10-K) -> Net-(U10-REF)
- U10 pad 2: Net-(Q6-S) -> Net-(U10-K)
- U13 pad 1: Net-(U13-K) -> Net-(U13-REF)
- U13 pad 2: Net-(Q8-S) -> Net-(U13-K)
- U15 pad 1: Net-(U15-K) -> Net-(U15-REF)
- U15 pad 2: Net-(Q10-S) -> Net-(U15-K)
- U17 pad 1: Net-(U17-K) -> Net-(U17-REF)
- U17 pad 2: Net-(Q13-S) -> Net-(U17-K)
- U19 pad 1: Net-(U19-K) -> Net-(U19-REF)
- U19 pad 2: U_BAT_1 -> Net-(U19-K)
- U20 pad 1: Net-(U20-K) -> Net-(U20-REF)
- U20 pad 2: U_BAT_0 -> Net-(U20-K)
Routing:
- net Net-(Q10-S): track 0.00 -> 27.9 mm, vias 0 -> 2
- net Net-(Q8-S): track 0.00 -> 27.8 mm, vias 0 -> 2
- net Net-(Q2-S): track 0.00 -> 27.7 mm, vias 0 -> 2
- net Net-(Q13-S): track 0.00 -> 27.7 mm, vias 0 -> 2
- net Net-(Q6-S): track 0.00 -> 27.6 mm, vias 0 -> 2
- net Net-(Q4-S): track 0.00 -> 27.6 mm, vias 0 -> 2
- net U_BAT_1: track 0.00 -> 26.7 mm, vias 0 -> 1
- net Net-(Q1-E): track 0.00 -> 19.7 mm, vias 0 -> 1
- net Net-(Q11-C): track 0.00 -> 14.7 mm, vias 0 -> 1
- net Net-(Q14-C): track 0.00 -> 14.6 mm, vias 0 -> 1
- net Net-(Q1-C): track 0.00 -> 14.6 mm, vias 0 -> 1
- net Net-(Q3-C): track 0.00 -> 14.4 mm, vias 0 -> 1
- net Net-(Q10-G): track 0.00 -> 14.4 mm, vias 0 -> 1
- net Net-(Q5-C): track 0.00 -> 14.4 mm, vias 0 -> 1
- net Net-(Q7-C): track 0.00 -> 14.1 mm, vias 0 -> 1
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- added copper zone on B.Cu, net Net-(Q11-B)
- added copper zone on B.Cu, net Net-(Q14-B)
- added copper zone on B.Cu, net Net-(Q16-B)
- added copper zone on B.Cu, net Net-(Q5-B)
- added copper zone on B.Cu, net Net-(Q9-B)
Other:
- board size 413.4 x 187.5 mm -> 379.5 x 118.1 mm

Commit message: 18.03.2025
Parts:
- U10, U13, U15, U17, U19, U20, U5, U8: value TL432DBZ -> TL431A
Changed lines of the file:
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@@
 			)
 		)
-		(property "Value" "TL432DBZ"
+		(property "Value" "TL431A"
 			(at 0 -2.4 90)
 			(layer "B.Fab")
@@
 			)
 		)
-		(property "Value" "TL432DBZ"
+		(property "Value" "TL431A"
 			(at 0 -2.4 90)
 			(layer "B.Fab")
@@
 			)
 		)
-		(property "Value" "TL432DBZ"
+		(property "Value" "TL431A"
 			(at 0 -2.4 90)
 			(layer "B.Fab")
@@
 			)
 		)
-		(property "Value" "TL432DBZ"
+		(property "Value" "TL431A"
 			(at 0 -2.4 90)
 			(layer "B.Fab")
@@
 			)
 		)
-		(property "Value" "TL432DBZ"
+		(property "Value" "TL431A"
 			(at 0 -2.4 90)
 			(layer "B.Fab")
@@
 			)
 		)
-		(property "Value" "TL432DBZ"
+		(property "Value" "TL431A"
 			(at 0 -2.4 90)
 			(layer "B.Fab")
@@
 			)
 		)
-		(property "Value" "TL432DBZ"
+		(property "Value" "TL431A"
 			(at 0 -2.4 90)
 			(layer "B.Fab")
@@
 			)
 		)
-		(property "Value" "TL432DBZ"
+		(property "Value" "TL431A"
 			(at 0 -2.4 90)
 			(layer "B.Fab")

Commit message: 22.03.2025
Parts:
- added H1: MountingHole, MountingHole:MountingHole_4.3mm_M4_Pad_Via, F.Cu at (236.8, 58.2)
- added J8: 430450800, Connector_Molex:Molex_Micro-Fit_3.0_43045-0800_2x04_P3.00mm_Horizontal, F.Cu at (177.7, 146.0)
- added J9: 430450800, Connector_Molex:Molex_Micro-Fit_3.0_43045-0800_2x04_P3.00mm_Horizontal, F.Cu at (151.7, 146.4)
- J3, L1, R3: moved to B.Cu
- J5: value 430451200 -> 430451000; footprint Connector_Molex:Molex_Micro-Fit_3.0_43045-1200_2x06_P3.00mm_Horizontal -> Connector_Molex:Molex_Micro-Fit_3.0_43045-1000_2x05_P3.00mm_Horizontal
- moved C23 340.1 mm to (215.0, 145.7)
- moved C24 340.1 mm to (215.0, 148.3)
- moved U11 306.7 mm to (225.4, 144.6)
- moved U2 275.0 mm to (183.2, 231.2), turned to 180 degrees
- moved C14 270.1 mm to (191.3, 234.2), turned to 90 degrees
- moved C15 267.6 mm to (189.9, 234.2), turned to 90 degrees
- moved L1 263.2 mm to (176.5, 231.1), turned to 180 degrees
- moved U18 257.0 mm to (188.2, 108.8)
- moved C13 256.8 mm to (176.5, 231.1), turned to 90 degrees
- moved J4 255.1 mm to (175.2, 227.2), turned to -90 degrees
- moved D1 255.0 mm to (172.9, 231.1)
- moved J3 254.1 mm to (167.0, 229.6), turned to -90 degrees
- moved U14 253.1 mm to (177.2, 108.6)
- moved U9 253.1 mm to (168.7, 108.6)
- moved R3 245.1 mm to (170.8, 224.6)
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Connections:
- D1 pad 1: CAN0+ -> CAN0-
- D1 pad 2: CAN0- -> CAN0+
- J5 pad 1: TERMO_0_OUT -> U_BAT_8
- J5 pad 10: unconnected-(J5-Pad10) -> U_BAT_0
- J5 pad 2: TERMO_1_OUT -> U_BAT_7
- J5 pad 3: TERMO_2_OUT -> U_BAT_6
- J5 pad 4: TERMO_3_OUT -> U_BAT_5
- J5 pad 5: TERMO_4_OUT -> U_BAT_4
- J5 pad 6: TERMO_5_OUT -> U_BAT_3
- J5 pad 7: TERMO_6_OUT -> U_BAT_2
- J5 pad 8: TERMO_7_OUT -> U_BAT_1
- R2 pad 1: NRST -> BOOT0
- R76 pad 1: Net-(U18-EN) -> unconnected-(R76-Pad1)
- R76 pad 2: 5V_ADC -> unconnected-(R76-Pad2)
- U1 pad 44: CAN1_STM32_TX -> CAN1_STM32_RX
- U1 pad 45: CAN1_STM32_RX -> CAN1_STM32_TX
- U1 pad 60: unconnected-(U1-BOOT0-Pad60) -> BOOT0
- U18 pad 5: SPI1_SCK_ADC -> unconnected-(U18-GND-Pad5)
- U18 pad 6: 5V_ADC -> unconnected-(U18-VO-Pad6)
- U18 pad 7: Net-(U18-EN) -> unconnected-(U18-EN-Pad7)
- U18 pad 8: 5V_ADC -> unconnected-(U18-VCC-Pad8)
Routing:
- net CAN0+: track 0.00 -> 22.7 mm
- net GND_CAN1: track 0.00 -> 11.6 mm
- net CAN0-: track 0.00 -> 9.19 mm
- net (no net): track 5.70 -> 0.00 mm
- net GND: track 17.4 -> 22.8 mm, vias 6 -> 8
- net 3v3: track 0.00 -> 5.05 mm, vias 0 -> 1
- net Net-(J4-Pin_1): track 0.00 -> 4.65 mm
- net Net-(U2-VCC2): track 0.00 -> 3.97 mm
- net 3V3: track 20.5 -> 17.0 mm, vias 5 -> 4
- net CAN0_ISO+: track 0.00 -> 1.63 mm, vias 0 -> 1
- net CAN0_ISO-: track 0.00 -> 1.55 mm, vias 0 -> 1
Other:
- board size 379.5 x 118.1 mm -> 379.5 x 253.7 mm

Commit message: 23.03.2025
Parts:
- R81: value 500 -> 180
- moved U14 452.1 mm to (-267.5, 27.0)
- moved U16 452.1 mm to (-298.3, 26.2)
- moved U18 452.1 mm to (-256.5, 27.2)
- moved C23 356.3 mm to (219.5, 502.0)
- moved C24 356.3 mm to (219.5, 504.5)
- moved J8 356.3 mm to (182.1, 502.2)
- moved J9 356.3 mm to (156.2, 502.7)
- moved U11 169.9 mm to (379.8, 73.6)
- moved U7 29.5 mm to (122.8, 81.2), turned to 90 degrees
- moved R_bal_8 26.6 mm to (144.8, 76.9)
- moved Q1 26.6 mm to (212.3, 85.0)
- moved Q11 26.6 mm to (161.3, 85.0)
- moved Q13 26.6 mm to (162.7, 81.5)
- moved Q2 26.6 mm to (213.8, 81.5)
- moved Q3 26.6 mm to (202.2, 85.0)
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Connections:
- C24 pad 1: 5V_ADC -> SPI1_SCK_ADC
- Q12 pad 1: 5V0 -> 3V3
- Q12 pad 2: Net-(Q12-S) -> SPI1_MISO
- Q12 pad 3: SPI1_MISO -> Net-(Q12-D)
- R100 pad 1: 5V_ADC -> SPI1_SCK_ADC
- R101 pad 1: 5V_ADC -> SPI1_SCK_ADC
- R102 pad 1: 5V_ADC -> SPI1_SCK_ADC
- R63 pad 1: Net-(Q12-S) -> Net-(Q12-D)
- R76 pad 1: unconnected-(R76-Pad1) -> SPI1_SCK_ADC
- R76 pad 2: unconnected-(R76-Pad2) -> Net-(U18-EN)
- R93 pad 1: 5V_ADC -> SPI1_SCK_ADC
- R94 pad 1: 5V_ADC -> SPI1_SCK_ADC
- R95 pad 1: 5V_ADC -> SPI1_SCK_ADC
- R97 pad 1: 5V_ADC -> SPI1_SCK_ADC
- R99 pad 1: 5V_ADC -> SPI1_SCK_ADC
- U11 pad 8: 5V_ADC -> SPI1_SCK_ADC
- U12 pad 1: 5V_ADC -> SPI1_SCK_ADC
- U12 pad 8: 5V_ADC -> SPI1_SCK_ADC
- U14 pad 5: GND -> U_BAT_0
- U16 pad 2: 5V_ADC -> SPI1_SCK_ADC
- U16 pad 6: Net-(Q12-S) -> Net-(Q12-D)
- U18 pad 5: unconnected-(U18-GND-Pad5) -> U_BAT_0
- U18 pad 7: unconnected-(U18-EN-Pad7) -> Net-(U18-EN)
- U18 pad 8: unconnected-(U18-VCC-Pad8) -> SPI1_SCK_ADC
- U21 pad 16: 5V_ADC -> SPI1_SCK_ADC
- U22 pad 1: 5V_ADC -> SPI1_SCK_ADC
- U22 pad 8: 5V_ADC -> SPI1_SCK_ADC
- U23 pad 8: 5V_ADC -> SPI1_SCK_ADC
- U6 pad 8: 5V_ADC -> SPI1_SCK_ADC
- U7 pad 16: 5V_ADC -> SPI1_SCK_ADC
- U9 pad 8: 5V_ADC -> SPI1_SCK_ADC
Routing:
- net U_BAT_8: track 1.46 -> 102.6 mm, vias 0 -> 1
- net U_BAT_7: track 1.46 -> 92.2 mm
- net U_BAT_6: track 1.46 -> 82.5 mm
- net U_BAT_5: track 1.46 -> 69.7 mm
- net U_BAT_4: track 1.46 -> 63.9 mm
- net U_BAT_3: track 1.46 -> 48.5 mm
- net U_BAT_2: track 1.46 -> 45.7 mm, vias 0 -> 1
- net U_BAT_1: track 26.7 -> 47.7 mm
Other:
- board size 379.5 x 253.7 mm -> 575.3 x 255.6 mm
