File: KiCad/BMS/BMS.kicad_pcb (KiCad board)
At the start: 4 copper layers, 575.3 x 255.6 mm, 186 parts, among them J1 PLS-6, J2 BH1,27-10-G, J3 430450400, J4 Conn_01x03, J5 430451000, J8 430450800, J9 430450800, Q1 PNP, Q10 NMOS, Q11 PNP, Q12 BSS138, Q13 NMOS, Q14 PNP, Q15 NMOS, Q16 PNP, Q17 NMOS, Q2 NMOS, Q3 PNP, Q4 NMOS, Q5 PNP, Q6 NMOS, Q7 PNP, Q8 NMOS, Q9 PNP, SW1 B3F1060, SW2 MSS-12D16, U1 STM32F405RGTx, U10 TL431A, U11 B0505MT, U12 MCP3201, U13 TL431A, U14 HCPL-0630, U15 TL431A, U16 HCPL-0600, U17 TL431A, U18 HCPL-0600, U19 TL431A, U2 ISO1050DUB, U20 TL431A, U21 74HC4051, U22 MCP3201, U23 HCPL-0630, U3 ST1S14PHR, U4 LDL1117S33R, U5 TL431A, U6 HCPL-0630, U7 74HC4051, U8 TL431A, U9 HCPL-0630, Y1 Crystal

Commit message: 25.03.2025
Parts:
- added R10: 3m, Resistor_SMD:R_0603_1608Metric, F.Cu at (145.0, 82.8)
- added R21: 3m, Resistor_SMD:R_0603_1608Metric, F.Cu at (155.2, 81.3)
- added R32: 3m, Resistor_SMD:R_0603_1608Metric, F.Cu at (165.1, 81.3)
- added R43: 3m, Resistor_SMD:R_0603_1608Metric, F.Cu at (175.8, 81.3)
- added R7: 1m, Resistor_SMD:R_0603_1608Metric, F.Cu at (145.0, 79.9)
- C22: renamed from C17; footprint Capacitor_THT:CP_Radial_D5.0mm_P2.00mm -> Capacitor_THT:CP_Radial_D6.3mm_P2.50mm
- R20: value 6m -> 3m
- R31: value 5m -> 2m
- R41: renamed from R42; value 4m -> 1m
- R9: value 7m -> 3m
- U11: renamed from U12; moved to B.Cu
- Y1: value Crystal -> Crystal KSE-7U08000MAB143ZA3
- moved R85 82.4 mm to (220.7, 71.8), turned to 90 degrees
- moved R87 81.8 mm to (220.6, 75.5), turned to 90 degrees
- moved R86 79.6 mm to (219.5, 76.3), turned to 0 degrees
- moved R84 78.1 mm to (218.7, 79.0), turned to 180 degrees
- moved Q16 78.0 mm to (217.8, 67.7), turned to 90 degrees
- moved U20 77.1 mm to (218.0, 71.7), turned to 90 degrees
- moved Q17 74.0 mm to (216.4, 71.3), turned to 90 degrees
- moved R82 73.2 mm to (215.4, 68.1), turned to 90 degrees
- moved R83 72.2 mm to (215.6, 71.7), turned to 90 degrees
- moved R8 72.1 mm to (144.7, 67.8), turned to 90 degrees
- moved R_bal_1 71.5 mm to (144.0, 75.4), turned to 180 degrees
- moved R15 70.6 mm to (145.0, 84.2), turned to 180 degrees
- moved R11 70.4 mm to (144.9, 71.5), turned to 90 degrees
- moved R9 69.9 mm to (145.0, 81.3)
- moved R_bal_8 69.9 mm to (214.7, 75.6), turned to 180 degrees
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- renumbered C9 to C10, C20 to C17, C21 to C18, C18 to C19, C19 to C20, C22 to C21, C10 to C9, D6 to D3, D7 to D4, D13 to D5, D14 to D6, J8 to J6, J9 to J7, R10 to R11, R11 to R12, R12 to R15, R15 to R16, R16 to R17, R17 to R18, R18 to R19, R21 to R22, R22 to R23, R23 to R24, R24 to R25, R25 to R26, R26 to R27, R27 to R28, R28 to R29, R29 to R30, R32 to R33, R33 to R34, R34 to R35, R35 to R36, R36 to R37, R37 to R38, R38 to R39, R39 to R40, R41 to R42, R43 to R44, R44 to R45, R45 to R46, R46 to R47, R47 to R48, R48 to R49, R51 to R50, R49 to R51, R57 to R52, R52 to R53, R53 to R54, R54 to R55, R55 to R56, R56 to R57, R65 to R60, R60 to R61, R68 to R65, R69 to R68, R70 to R69, R71 to R70, R72 to R71, R75 to R72, R79 to R74, R77 to R75, R78 to R76, R76 to R77, R80 to R78, R81 to R79, R7 to R8, R82 to R80, R83 to R81, R84 to R82, R86 to R83, R87 to R84, R88 to R85, R89 to R86, R90 to R87, R91 to R88, R92 to R89, R93 to R90, R94 to R91, R95 to R92, R96 to R93, R97 to R94, R98 to R95, R99 to R96, R100 to R97, R101 to R98, R102 to R99, U11 to U12
Connections:
- C24 pad 1: SPI1_SCK_ADC -> 5V_ADC
- J5 pad 2: U_BAT_7 -> U_BAT_6
- J5 pad 3: U_BAT_6 -> U_BAT_4
- J5 pad 4: U_BAT_5 -> U_BAT_2
- J5 pad 5: U_BAT_4 -> U_BAT_0
- J5 pad 6: U_BAT_3 -> U_BAT_7
- J5 pad 7: U_BAT_2 -> U_BAT_5
- J5 pad 8: U_BAT_1 -> U_BAT_3
- J5 pad 9: unconnected-(J5-Pad9) -> U_BAT_1
- Q1 pad 3: Net-(Q1-E) -> U_BAT_8
- Q10 pad 3: Net-(Q10-S) -> U_BAT_3
- Q11 pad 3: Net-(Q10-S) -> U_BAT_3
- Q13 pad 3: Net-(Q13-S) -> U_BAT_2
- Q14 pad 3: Net-(Q13-S) -> U_BAT_2
- Q2 pad 3: Net-(Q2-S) -> U_BAT_7
- Q3 pad 3: Net-(Q2-S) -> U_BAT_7
- Q4 pad 3: Net-(Q4-S) -> U_BAT_6
- Q5 pad 3: Net-(Q4-S) -> U_BAT_6
- Q6 pad 3: Net-(Q6-S) -> U_BAT_5
- Q7 pad 3: Net-(Q6-S) -> U_BAT_5
- Q8 pad 3: Net-(Q8-S) -> U_BAT_4
- Q9 pad 3: Net-(Q8-S) -> U_BAT_4
- R12 pad 2: Net-(Q1-E) -> U_BAT_8
- R15 pad 2: U_BAT_8 -> U_MES_8
- R17 pad 1: Net-(Q2-S) -> U_BAT_7
- R18 pad 1: Net-(Q2-S) -> U_BAT_7
- R19 pad 2: Net-(Q2-S) -> U_BAT_7
- R20 pad 1: U_BAT_7 -> Net-(R20-Pad1)
- R20 pad 2: Net-(Q2-S) -> U_BAT_7
- R23 pad 2: Net-(Q2-S) -> U_BAT_7
- R24 pad 2: U_BAT_7 -> U_MES_7
- R27 pad 1: Net-(Q4-S) -> U_BAT_6
- R28 pad 1: Net-(Q4-S) -> U_BAT_6
- R30 pad 2: Net-(Q4-S) -> U_BAT_6
- R31 pad 1: U_BAT_6 -> Net-(R31-Pad1)
- R31 pad 2: Net-(Q4-S) -> U_BAT_6
- R34 pad 2: Net-(Q4-S) -> U_BAT_6
- R35 pad 2: U_BAT_6 -> U_MES_6
- R37 pad 1: Net-(Q6-S) -> U_BAT_5
- R38 pad 1: Net-(Q6-S) -> U_BAT_5
- R40 pad 2: Net-(Q6-S) -> U_BAT_5
- R41 pad 1: U_BAT_5 -> Net-(R41-Pad1)
- R41 pad 2: Net-(Q6-S) -> U_BAT_5
- R45 pad 2: Net-(Q6-S) -> U_BAT_5
- R46 pad 2: U_BAT_5 -> U_MES_5
- R48 pad 1: Net-(Q8-S) -> U_BAT_4
- R49 pad 1: Net-(Q8-S) -> U_BAT_4
- R50 pad 1: U_BAT_4 -> U_MES_4
- R50 pad 2: Net-(Q8-S) -> U_BAT_4
- R51 pad 2: Net-(Q8-S) -> U_BAT_4
- R52 pad 2: U_BAT_4 -> U_MES_4
- R55 pad 2: Net-(Q8-S) -> U_BAT_4
- R58 pad 1: Net-(Q10-S) -> U_BAT_3
- R59 pad 1: Net-(Q10-S) -> U_BAT_3
- R60 pad 1: U_BAT_3 -> U_MES_3
- R60 pad 2: Net-(Q10-S) -> U_BAT_3
- R61 pad 2: Net-(Q10-S) -> U_BAT_3
- R65 pad 2: U_BAT_3 -> U_MES_3
- R67 pad 2: Net-(Q10-S) -> U_BAT_3
- R70 pad 1: Net-(Q13-S) -> U_BAT_2
- R71 pad 1: Net-(Q13-S) -> U_BAT_2
- R72 pad 1: U_BAT_2 -> U_MES_2
- R72 pad 2: Net-(Q13-S) -> U_BAT_2
- R73 pad 2: Net-(Q13-S) -> U_BAT_2
- R74 pad 2: U_BAT_2 -> U_MES_2
- R76 pad 2: Net-(Q13-S) -> U_BAT_2
- R77 pad 1: SPI1_SCK_ADC -> 5V_ADC
- R8 pad 2: Net-(Q1-E) -> U_BAT_8
- R9 pad 1: U_BAT_8 -> Net-(R10-Pad1)
- R9 pad 2: Net-(Q1-E) -> Net-(R7-Pad2)
- R90 pad 1: SPI1_SCK_ADC -> 5V_ADC
- R91 pad 1: SPI1_SCK_ADC -> 5V_ADC
- R92 pad 1: SPI1_SCK_ADC -> 5V_ADC
- R94 pad 1: SPI1_SCK_ADC -> 5V_ADC
- R96 pad 1: SPI1_SCK_ADC -> 5V_ADC
- R97 pad 1: SPI1_SCK_ADC -> 5V_ADC
- R98 pad 1: SPI1_SCK_ADC -> 5V_ADC
- R99 pad 1: SPI1_SCK_ADC -> 5V_ADC
- R_bal_1 pad 2: Net-(Q1-E) -> U_BAT_8
- R_bal_2 pad 2: Net-(Q2-S) -> U_BAT_7
- R_bal_3 pad 2: Net-(Q4-S) -> U_BAT_6
- R_bal_4 pad 2: Net-(Q6-S) -> U_BAT_5
- R_bal_5 pad 2: Net-(Q8-S) -> U_BAT_4
- R_bal_6 pad 2: Net-(Q10-S) -> U_BAT_3
- R_bal_7 pad 2: Net-(Q13-S) -> U_BAT_2
- U10 pad 3: Net-(Q6-S) -> U_BAT_5
- U11 pad 1: SPI1_SCK_ADC -> 5V_ADC
- U11 pad 8: SPI1_SCK_ADC -> 5V_ADC
- U12 pad 8: SPI1_SCK_ADC -> 5V_ADC
- U13 pad 3: Net-(Q8-S) -> U_BAT_4
- U15 pad 3: Net-(Q10-S) -> U_BAT_3
- U16 pad 2: SPI1_SCK_ADC -> 5V_ADC
- U17 pad 3: Net-(Q13-S) -> U_BAT_2
- U18 pad 6: unconnected-(U18-VO-Pad6) -> SPI1_SCK_ADC
- U18 pad 8: SPI1_SCK_ADC -> 5V_ADC
- U21 pad 16: SPI1_SCK_ADC -> 5V_ADC
- U22 pad 1: SPI1_SCK_ADC -> 5V_ADC
- U22 pad 8: SPI1_SCK_ADC -> 5V_ADC
- U23 pad 8: SPI1_SCK_ADC -> 5V_ADC
- U5 pad 3: Net-(Q2-S) -> U_BAT_7
- U6 pad 8: SPI1_SCK_ADC -> 5V_ADC
- U7 pad 1: U_BAT_4 -> U_BAT_1
- U7 pad 12: U_BAT_5 -> U_MES_5
- U7 pad 13: U_BAT_8 -> U_MES_6
- U7 pad 14: U_BAT_7 -> U_MES_7
- U7 pad 15: U_BAT_6 -> U_MES_8
- U7 pad 16: SPI1_SCK_ADC -> 5V_ADC
- U7 pad 2: U_BAT_2 -> U_MES_2
- U7 pad 4: U_BAT_1 -> U_MES_3
- U7 pad 5: U_BAT_3 -> U_MES_4
- U8 pad 3: Net-(Q4-S) -> U_BAT_6
- U9 pad 8: SPI1_SCK_ADC -> 5V_ADC
Routing:
- net U_BAT_1: track 47.7 -> 104.7 mm
- net U_BAT_8: track 102.6 -> 50.7 mm
- net U_BAT_7: track 92.2 -> 47.4 mm, vias 0 -> 2
- net U_BAT_6: track 82.5 -> 42.9 mm, vias 0 -> 2
- net U_BAT_5: track 69.7 -> 31.3 mm, vias 0 -> 2
- net U_MES_8: track 0.00 -> 37.4 mm
- net Net-(Q10-S): track 27.9 -> 0.00 mm, vias 2 -> 0
- net Net-(Q8-S): track 27.8 -> 0.00 mm, vias 2 -> 0
- net Net-(Q2-S): track 27.7 -> 0.00 mm, vias 2 -> 0
- net Net-(Q13-S): track 27.7 -> 0.00 mm, vias 2 -> 0
- net Net-(Q6-S): track 27.6 -> 0.00 mm, vias 2 -> 0
- net Net-(Q4-S): track 27.6 -> 0.00 mm, vias 2 -> 0
- net U_BAT_4: track 63.9 -> 38.0 mm, vias 0 -> 2
- net U_MES_7: track 0.00 -> 25.8 mm
- net U_MES_2: track 0.00 -> 24.8 mm
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- added copper zone on B.Cu, net Net-(Q1-B)
- added copper zone on B.Cu, net Net-(Q3-B)
- added copper zone on B.Cu, net Net-(Q7-B)

Commit message: 27.03.2025
Parts:
- C10, C11, C12, C13, C14, C15, C2, C21, C23, C24, C3, C4, C5, C6, C7, C8, C9, D1, J1, J2, J4, JP1, L2, R1, R2, R5, SW1, SW2, U1, U14, U18, U2, U22, U23, Y1: moved to B.Cu
- J3, L1, R3: moved to F.Cu
- moved U16 500.8 mm to (198.1, 92.3)
- moved U14 470.4 mm to (197.9, 95.2), turned to 180 degrees
- moved U18 458.6 mm to (197.8, 89.8), turned to 180 degrees
- moved C24 406.0 mm to (164.9, 102.2), turned to -90 degrees
- moved C23 404.5 mm to (157.9, 102.2), turned to -90 degrees
- moved J7 391.5 mm to (174.4, 111.6)
- moved J6 391.4 mm to (203.7, 111.5)
- moved H1 337.3 mm to (-95.6, 115.3)
- moved C1 287.3 mm to (264.5, 88.3), turned to -90 degrees
- moved J2 285.5 mm to (260.1, 103.9)
- moved J1 283.9 mm to (264.8, 107.7)
- moved R39 281.2 mm to (161.1, 152.6)
- moved R42 281.2 mm to (161.1, 160.1)
- moved R77 281.2 mm to (173.1, 147.6)
- moved R79 281.2 mm to (173.1, 160.1)
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Connections:
- C23 pad 1: 5V -> 5V0
- U12 pad 13: 5V -> 5V0
- U12 pad 14: 5V -> 5V0
- U21 pad 1: TERMO_3_OUT -> TERMO_3_IN
- U21 pad 12: TERMO_4_OUT -> TERMO_4_IN
- U21 pad 13: TERMO_7_OUT -> TERMO_7_IN
- U21 pad 14: TERMO_6_OUT -> TERMO_6_IN
- U21 pad 15: TERMO_5_OUT -> TERMO_5_IN
- U21 pad 2: TERMO_1_OUT -> TERMO_1_IN
- U21 pad 4: TERMO_0_OUT -> TERMO_0_IN
- U21 pad 5: TERMO_2_OUT -> TERMO_2_IN
Routing:
- net NRST: track 0.00 -> 30.9 mm, vias 0 -> 1
- net DEBUG_SWD_IO: track 0.00 -> 29.9 mm, vias 0 -> 1
- net GND: track 22.8 -> 44.2 mm, vias 8 -> 14
- net 3V3: track 17.0 -> 30.5 mm, vias 4 -> 8
- net U_BAT_1: track 104.7 -> 91.6 mm
- net U_BAT_0: track 7.79 -> 20.0 mm, vias 5 -> 10
- net 5V_ADC: track 0.00 -> 10.5 mm, vias 0 -> 2
- net MPL_VOLT_2_5V: track 0.00 -> 9.04 mm
- net 5V0: track 0.00 -> 8.88 mm, vias 0 -> 3
- net DEBUG_SWD_SWO: track 0.00 -> 8.11 mm
- net MPL_VOLT_1_5V: track 0.00 -> 7.35 mm
- net Net-(D2-K): track 0.00 -> 7.15 mm, vias 0 -> 1
- net U_MEASURE: track 0.00 -> 5.68 mm, vias 0 -> 1
- net Net-(U3-FB): track 0.00 -> 5.33 mm, vias 0 -> 1
- net U_BAT_2: track 54.0 -> 50.0 mm
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- added copper zone on B.Cu, net 5V0
- added copper zone on F.Cu, net 5V0
- added copper zone on B.Cu, net GND
- added copper zone on B.Cu, net U_BAT_0
- added copper zone on F.Cu, net U_BAT_0
Other:
- board size 575.3 x 255.6 mm -> 368.5 x 89.3 mm

Commit message: 30.03.2025
Parts:
- removed D5, D6: BZX384xxxx, Diode_SMD:D_SOD-323_HandSoldering
- removed R88, R89: R, Resistor_SMD:R_0603_1608Metric
- added D7: BZX384-C4V7, Diode_SMD:D_SOD-323_HandSoldering, F.Cu at (171.1, 109.4)
- added D8: BZX384-C4V7, Diode_SMD:D_SOD-323_HandSoldering, F.Cu at (171.1, 112.3)
- added H2: MountingHole, MountingHole:MountingHole_3.2mm_M3_Pad_Via, F.Cu at (245.6, 52.5)
- added H3: MountingHole, MountingHole:MountingHole_3.2mm_M3_Pad_Via, F.Cu at (245.6, 44.4)
- added H4: MountingHole, MountingHole:MountingHole_3.2mm_M3_Pad_Via, F.Cu at (245.3, 61.2)
- added H5: MountingHole, MountingHole:MountingHole_3.2mm_M3_Pad_Via, F.Cu at (245.3, 69.2)
- added H6: MountingHole, MountingHole:MountingHole_3.2mm_M3_Pad_Via, F.Cu at (245.3, 77.1)
- added J8: 430450400, Connector_Molex:Molex_Micro-Fit_3.0_43045-0400_2x02_P3.00mm_Horizontal, F.Cu at (132.9, 84.8)
- C1, R77, R79: moved to B.Cu
- D3, D4: value BZX384xxxx -> BZX384-C4V7
- H1: footprint MountingHole:MountingHole_4.3mm_M4_Pad_Via -> MountingHole:MountingHole_3.2mm_M3_Pad_Via
- SW1, U23: moved to F.Cu
- moved H1 328.2 mm to (227.3, 56.8)
- moved R63 279.7 mm to (-5.84, -70.7)
- moved R69 279.7 mm to (-5.84, -55.6)
- moved R64 279.7 mm to (-5.84, -68.1)
- moved R93 279.7 mm to (-9.57, -72.8)
- moved R95 279.7 mm to (-9.57, -67.8)
- moved R39 78.3 mm to (197.4, 83.2), turned to 90 degrees
- moved J2 77.8 mm to (200.5, 54.0), turned to 90 degrees
- moved R29 75.6 mm to (189.5, 94.3), turned to 180 degrees
- moved R16 74.6 mm to (189.5, 100.0), turned to 180 degrees
- moved J1 72.6 mm to (217.3, 52.8), turned to 90 degrees
- moved R14 69.6 mm to (189.5, 98.3), turned to 180 degrees
- moved C10 69.1 mm to (191.8, 91.9), turned to -90 degrees
- moved R79 67.2 mm to (186.6, 94.3), turned to 90 degrees
- moved R26 67.0 mm to (189.5, 96.5), turned to 180 degrees
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Connections:
- D3 pad 1: Net-(D3-K) -> 5V_ADC
- D3 pad 2: Net-(D3-A) -> U_MEASURE_CLR
- D4 pad 1: Net-(D4-K) -> U_MEASURE_CLR
- D4 pad 2: Net-(D3-A) -> U_BAT_0
- R39 pad 1: Net-(D3-K) -> U_MEASURE_CLR
- R42 pad 1: Net-(D4-K) -> T_MEASURE_CLR
- R42 pad 2: U_BAT_0 -> T_MEASURE
- U11 pad 2: U_MEASURE -> U_MEASURE_CLR
- U22 pad 2: T_MEASURE -> T_MEASURE_CLR
Routing:
- net NRST: track 30.9 -> 0.00 mm, vias 1 -> 0
- net DEBUG_SWD_IO: track 29.9 -> 0.00 mm, vias 1 -> 0
- net SPI1_SCK_ADC: track 0.00 -> 18.2 mm
- net GND: track 44.2 -> 32.1 mm, vias 14 -> 12
- net MPL_VOLT_0_5V: track 0.00 -> 10.3 mm, vias 1 -> 2
- net MPL_TEMP_0_5V: track 0.00 -> 8.41 mm, vias 0 -> 2
- net DEBUG_SWD_SWO: track 8.11 -> 0.00 mm
- net 5V_ADC: track 10.5 -> 18.6 mm, vias 2 -> 6
- net U_MEASURE: track 5.68 -> 0.00 mm, vias 1 -> 0
- net DEBUG_SWD_CLK: track 3.38 -> 0.00 mm
- net U_BAT_0: track 20.0 -> 23.0 mm, vias 10 -> 14
- net BOOT0: track 3.00 -> 0.00 mm
- net Net-(J2-Pin_1): track 2.60 -> 0.00 mm
- net Net-(U18-C): track 0.00 -> 2.03 mm
- net Net-(U18-EN): track 0.00 -> 1.96 mm
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- added copper zone on F.Cu, net 5V_ADC
Other:
- board size 368.5 x 89.3 mm -> 127.2 x 82.4 mm
