File: KiCad/BMS/BMS.kicad_pcb (KiCad board)
At the start: 4 copper layers, 127.2 x 82.4 mm, 195 parts, among them J1 PLS-6, J2 BH1,27-10-G, J3 430450400, J4 Conn_01x03, J5 430451000, J6 430450800, J7 430450800, J8 430450400, Q1 PNP, Q10 NMOS, Q11 PNP, Q12 BSS138, Q13 NMOS, Q14 PNP, Q15 NMOS, Q16 PNP, Q17 NMOS, Q2 NMOS, Q3 PNP, Q4 NMOS, Q5 PNP, Q6 NMOS, Q7 PNP, Q8 NMOS, Q9 PNP, SW1 B3F1060, SW2 MSS-12D16, U1 STM32F405RGTx, U10 TL431A, U11 MCP3201, U12 B0505MT, U13 TL431A, U14 HCPL-0630, U15 TL431A, U16 HCPL-0600, U17 TL431A, U18 HCPL-0600, U19 TL431A, U2 ISO1050DUB, U20 TL431A, U21 74HC4051, U22 MCP3201, U23 HCPL-0630, U3 ST1S14PHR, U4 LDL1117S33R, U5 TL431A, U6 HCPL-0630, U7 74HC4051, U8 TL431A, U9 HCPL-0630, Y1 Crystal KSE-7U08000MAB143ZA3

Commit message: rough routing is complete (04.04.2025)
Parts:
- removed R2: 10k, Resistor_SMD:R_0603_1608Metric
- removed SW2: MSS-12D16, user:MSS-12D16
- added C16: 4u7, Capacitor_SMD:C_0603_1608Metric, B.Cu at (137.6, 59.9)
- added C17: 10u, Capacitor_SMD:C_0603_1608Metric, F.Cu at (146.3, 60.0)
- added U3: B0505MT, user:B0505MT, F.Cu at (140.8, 60.0)
- C1: moved to F.Cu
- C24: renamed from C22; moved to B.Cu
- R39: moved to B.Cu
- R52: renamed from R53; moved to B.Cu
- R55: renamed from R56; moved to B.Cu
- R68: renamed from R69; moved to B.Cu
- R87: renamed from R42; moved to B.Cu
- U15: renamed from U14; moved to F.Cu
- U24: renamed from U23; moved to B.Cu
- moved R62 261.2 mm to (191.4, 100.6)
- moved R63 255.8 mm to (188.0, 98.9)
- moved R68 245.2 mm to (182.1, 101.9)
- moved R91 242.9 mm to (170.3, 90.4), turned to 90 degrees
- moved R93 236.8 mm to (169.3, 87.4)
- moved H3 113.9 mm to (132.1, 54.4), turned to 90 degrees
- moved H6 57.6 mm to (243.6, 19.6), turned to 90 degrees
- moved H5 50.5 mm to (235.7, 19.6), turned to 90 degrees
- moved H4 45.2 mm to (227.7, 19.6), turned to 90 degrees
- moved H1 44.9 mm to (252.8, 19.8), turned to 90 degrees
- moved C6 39.7 mm to (204.6, 99.2), turned to 0 degrees
- moved R87 33.4 mm to (160.7, 83.2), turned to -90 degrees
- moved J2 31.5 mm to (225.0, 73.8), turned to 0 degrees
- moved J3 30.7 mm to (164.4, 60.0), turned to 0 degrees
- moved U24 30.5 mm to (174.6, 88.9), turned to 0 degrees
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- renumbered C16 to C18, C17 to C19, C18 to C20, C19 to C21, C20 to C22, C21 to C23, C23 to C25, C24 to C26, D8 to D5, D7 to D6, J8 to J5, J5 to J6, J6 to J7, J7 to J8, R43 to R42, R44 to R43, R45 to R44, R46 to R45, R47 to R46, R48 to R47, R49 to R48, R50 to R49, R51 to R50, R52 to R51, R54 to R53, R55 to R54, R57 to R56, R58 to R57, R59 to R58, R60 to R59, R61 to R60, R62 to R61, R63 to R62, R64 to R63, R65 to R64, R66 to R65, R67 to R66, R68 to R67, R70 to R69, R71 to R70, R72 to R71, R73 to R72, R74 to R73, R75 to R74, R76 to R75, R77 to R76, R78 to R77, R79 to R78, R80 to R79, R81 to R80, R82 to R81, R83 to R82, R84 to R83, R85 to R84, R86 to R85, R87 to R86, R90 to R88, R91 to R89, R92 to R90, R93 to R91, R94 to R92, R95 to R93, R96 to R94, R97 to R95, R98 to R96, R99 to R97, U9 to U10, U10 to U11, U11 to U12, U12 to U13, U13 to U14, U15 to U16, U16 to U17, U17 to U18, U18 to U19, U19 to U20, U20 to U21, U21 to U23, U3 to U4, U4 to U5, U5 to U6, U6 to U7, U7 to U8, U8 to U9
Connections:
- net Net-(U2-VCC2) renamed 5V_CAN
- C13 pad 2: GND_CAN1 -> GND_CAN
- D1 pad 3: GND_CAN1 -> GND_CAN
- J3 pad 1: GND_CAN1 -> CAN0-
- J3 pad 2: GND_CAN1 -> GND_CAN
- J3 pad 3: CAN0- -> CAN0+
- J3 pad 4: CAN0+ -> GND_CAN
- J7 pad 1: TERMO_0_OUT -> TERMO_0
- J7 pad 2: TERMO_1_OUT -> TERMO_1
- J7 pad 3: TERMO_2_OUT -> TERMO_2
- J7 pad 4: TERMO_3_OUT -> TERMO_3
- J8 pad 1: TERMO_4_OUT -> TERMO_4
- J8 pad 2: TERMO_5_OUT -> TERMO_5
- J8 pad 3: TERMO_6_OUT -> TERMO_6
- J8 pad 4: TERMO_7_OUT -> TERMO_7
- R88 pad 2: TERMO_0_IN -> TERMO_0
- R89 pad 2: TERMO_1_IN -> TERMO_1
- R90 pad 2: TERMO_2_IN -> TERMO_2
- R92 pad 2: TERMO_3_IN -> TERMO_3
- R94 pad 2: TERMO_4_IN -> TERMO_4
- R95 pad 2: TERMO_5_IN -> TERMO_5
- R96 pad 2: TERMO_6_IN -> TERMO_6
- R97 pad 2: TERMO_7_IN -> TERMO_7
- U1 pad 57: unconnected-(U1-PB5-Pad57) -> MPL_TEMP_2_3V3
- U1 pad 58: unconnected-(U1-PB6-Pad58) -> MPL_TEMP_1_3V3
- U1 pad 59: unconnected-(U1-PB7-Pad59) -> MPL_TEMP_0_3V3
- U2 pad 5: GND_CAN1 -> GND_CAN
- U23 pad 1: TERMO_3_IN -> TERMO_3
- U23 pad 12: TERMO_4_IN -> TERMO_4
- U23 pad 13: TERMO_7_IN -> TERMO_7
- U23 pad 14: TERMO_6_IN -> TERMO_6
- U23 pad 15: TERMO_5_IN -> TERMO_5
- U23 pad 2: TERMO_1_IN -> TERMO_1
- U23 pad 4: TERMO_0_IN -> TERMO_0
- U23 pad 5: TERMO_2_IN -> TERMO_2
Routing:
- net CAN1_STM32_TX: track 0.00 -> 111.4 mm, vias 0 -> 5
- net CAN1_STM32_RX: track 0.00 -> 110.4 mm, vias 0 -> 4
- net NRST: track 0.00 -> 89.2 mm, vias 0 -> 2
- net TERMO_0: track 0.00 -> 75.3 mm, vias 0 -> 2
- net DEBUG_SWD_CLK: track 0.00 -> 74.7 mm, vias 0 -> 1
- net DEBUG_SWD_SWO: track 0.00 -> 72.0 mm
- net TERMO_1: track 0.00 -> 70.6 mm, vias 0 -> 3
- net TERMO_3: track 0.00 -> 67.2 mm, vias 0 -> 2
- net TERMO_2: track 0.00 -> 65.3 mm, vias 0 -> 2
- net MPL_TEMP_2_3V3: track 0.00 -> 55.2 mm, vias 0 -> 1
- net TERMO_4: track 0.00 -> 54.8 mm, vias 0 -> 2
- net TERMO_7: track 0.00 -> 52.5 mm, vias 0 -> 4
- net MPL_TEMP_1_3V3: track 0.00 -> 49.4 mm, vias 0 -> 1
- net TERMO_6: track 0.00 -> 44.1 mm, vias 0 -> 3
- net DEBUG_SWD_IO: track 0.00 -> 42.0 mm
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- added copper zone on B.Cu, net 5V_ADC
- added copper zone on F.Cu, net GND_CAN
- added copper zone on F.Cu, net NRST
- added copper zone on F.Cu, net Net-(U24-C2)
Other:
- board size 127.2 x 82.4 mm -> 129.3 x 93.6 mm

Commit message: 08.04.2025
Parts:
- removed U15: HCPL-0630, Package_SO:SOIC-8_3.9x4.9mm_P1.27mm
- moved C4 0.89 mm to (213.0, 84.4), turned to 0 degrees
- moved R61 0.75 mm to (191.4, 102.7), turned to 0 degrees
Connections:
- C19 pad 2: 5V0 -> 3V3
- C20 pad 2: 3V3 -> 5V0
- U5 pad 2: 5V0 -> 3V3
- U5 pad 3: 3V3 -> 5V0
Routing:
- net SPI1_SCK: track 3.66 -> 28.0 mm, vias 1 -> 2
- net GND_CAN: track 10.8 -> 18.5 mm, vias 1 -> 2
- net 3V3: track 40.4 -> 43.0 mm, vias 14 -> 15
- net DEBUG_SWD_CLK: track 74.7 -> 72.3 mm
- net TERMO_0: track 75.3 -> 73.7 mm
- net 5V_ADC: track 28.7 -> 30.0 mm, vias 9 -> 10
- net 5V0: track 21.6 -> 20.3 mm, vias 7 -> 5
- net SPI1_CS_1: track 15.5 -> 14.3 mm
- net 5V_CAN: track 7.48 -> 8.05 mm
- net SPI1_MISO: track 28.4 -> 29.0 mm
- added copper zone on In2.Cu, net GND
