File: KiCad/BMS/BMS.kicad_pcb (KiCad board)
At the start: 4 copper layers, 129.3 x 93.6 mm, 196 parts, among them J1 PLS-6, J2 BH1,27-10-G, J3 430450400, J4 Conn_01x03, J5 430450400, J6 430451000, J7 430450800, J8 430450800, Q1 PNP, Q10 NMOS, Q11 PNP, Q12 BSS138, Q13 NMOS, Q14 PNP, Q15 NMOS, Q16 PNP, Q17 NMOS, Q2 NMOS, Q3 PNP, Q4 NMOS, Q5 PNP, Q6 NMOS, Q7 PNP, Q8 NMOS, Q9 PNP, SW1 B3F1060, U1 STM32F405RGTx, U10 HCPL-0630, U11 TL431A, U12 MCP3201, U13 B0505MT, U14 TL431A, U15 HCPL-0630, U16 TL431A, U17 HCPL-0600, U18 TL431A, U19 HCPL-0600, U2 ISO1050DUB, U20 TL431A, U21 TL431A, U22 MCP3201, U23 74HC4051, U24 HCPL-0630, U3 B0505MT, U4 ST1S14PHR, U5 LDL1117S33R, U6 TL431A, U7 HCPL-0630, U8 74HC4051, U9 TL431A, Y1 Crystal KSE-7U08000MAB143ZA3

Commit message: 18.04.2025_final
Parts:
- removed the H1 at (252.8, 19.8)
- removed H6: MountingHole, MountingHole:MountingHole_3.2mm_M3_Pad_Via
- C1, R62, R90, R92, U17: moved to B.Cu
- R51, R54: moved to F.Cu
- moved H4 133.1 mm to (132.4, 103.5)
- moved H3 83.9 mm to (227.4, 103.5)
- moved R92 26.4 mm to (192.5, 99.9), turned to 180 degrees
- moved R90 23.0 mm to (192.5, 96.4), turned to 180 degrees
- moved R5 14.4 mm to (157.2, 84.2), turned to 90 degrees
- moved U24 14.2 mm to (186.2, 97.1), turned to 180 degrees
- moved R13 14.0 mm to (174.4, 100.0), turned to 90 degrees
- moved U22 13.3 mm to (170.5, 91.9)
- moved R67 13.0 mm to (178.6, 89.4), turned to 90 degrees
- moved C21 12.0 mm to (144.3, 85.4), turned to 90 degrees
- moved C18 11.9 mm to (155.2, 89.7), turned to -90 degrees
- moved R62 11.3 mm to (176.7, 99.8), turned to 180 degrees
- moved R3 11.2 mm to (152.7, 81.4), turned to 180 degrees
- moved R61 11.1 mm to (180.4, 102.5), turned to -90 degrees
- moved R15 10.2 mm to (179.0, 100.0), turned to 90 degrees
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- renumbered H2 to H1, H3 to H2, H4 to H3, H5 to H4, R93 to R87, R94 to R88, R95 to R89, R96 to R91, R87 to R93, R88 to R94, R91 to R95, R89 to R96
Connections:
- R87 pad 2: TERMO_4 -> TERMO_2
- R88 pad 2: TERMO_5 -> TERMO_0
- R89 pad 2: TERMO_6 -> TERMO_1
- R91 pad 2: TERMO_7 -> TERMO_3
- R93 pad 2: TERMO_0 -> TERMO_4
- R94 pad 2: TERMO_1 -> TERMO_5
- R95 pad 2: TERMO_3 -> TERMO_6
- R96 pad 2: TERMO_2 -> TERMO_7
- U1 pad 15: unconnected-(U1-PA1-Pad15) -> SPI1_CS_2
- U23 pad 1: TERMO_3 -> TERMO_6
- U23 pad 12: TERMO_4 -> TERMO_2
- U23 pad 13: TERMO_7 -> TERMO_3
- U23 pad 14: TERMO_6 -> TERMO_1
- U23 pad 15: TERMO_5 -> TERMO_0
- U23 pad 2: TERMO_1 -> TERMO_5
- U23 pad 4: TERMO_0 -> TERMO_4
- U23 pad 5: TERMO_2 -> TERMO_7
Routing:
- net MPL_TEMP_2_3V3: track 57.9 -> 17.3 mm, vias 1 -> 2
- net MPL_TEMP_1_3V3: track 51.3 -> 16.2 mm, vias 1 -> 0
- net DEBUG_SWD_IO: track 42.0 -> 74.1 mm, vias 0 -> 3
- net MPL_VOLT_1_5V: track 7.35 -> 32.7 mm, vias 0 -> 2
- net TERMO_0: track 73.6 -> 96.9 mm, vias 2 -> 1
- net T_MEASURE_CLR: track 33.5 -> 11.6 mm, vias 0 -> 2
- net MPL_TEMP_0_3V3: track 21.4 -> 39.6 mm
- net TERMO_1: track 73.7 -> 90.5 mm, vias 3 -> 1
- net MPL_TEMP_2_5V: track 3.12 -> 18.7 mm
- net MPL_TEMP_1_5V: track 5.19 -> 20.0 mm
- net TERMO_2: track 64.7 -> 78.1 mm, vias 0 -> 2
- net MPL_VOLT_0_3V3: track 28.4 -> 41.5 mm
- net 5V0: track 22.3 -> 10.8 mm, vias 6 -> 8
- net SPI1_SCK: track 30.1 -> 18.7 mm
- net MPL_VOLT_2_5V: track 9.04 -> 19.8 mm
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- added copper zone on In1.Cu, net 24V0
- added copper zone on In1.Cu, net 5V0
- added copper zone on In1.Cu, net 5V_CAN
- added copper zone on In2.Cu, net GND_CAN
- added copper zone on In2.Cu, net U_BAT_0
- added copper zone on B.Cu, net U_BAT_3
- added copper zone on B.Cu, net U_BAT_4
- added copper zone on B.Cu, net U_BAT_7
- removed copper zone on In2.Cu, net 3V3
- removed copper zone on B.Cu, net 5V_ADC
- removed copper zone on F.Cu, net Net-(U24-C2)
Other:
- board size 129.3 x 93.6 mm -> 103 x 57 mm

Commit message: 19.04.2025
Parts:
- added R2: 10k, Resistor_SMD:R_0603_1608Metric, F.Cu at (205.0, 97.3)
- added R6: 220, Resistor_SMD:R_0603_1608Metric, F.Cu at (104.1, 88.9)
- C21: renamed from C23; value C -> 150p
- L2: value 8u5 -> 6.8
- R4: renamed from R3; value 47k -> 10k
- R7: renamed from R5; value 2k7 -> 3k
- moved R11 1.11 mm to (148.8, 79.0), turned to 90 degrees
- moved R16 1.09 mm to (150.2, 79.0), turned to -90 degrees
- renumbered C21 to C19, C22 to C20, C19 to C22, C20 to C23, R8 to R10, R9 to R11, R10 to R12, R11 to R13, R12 to R14, R13 to R15, R14 to R16, R15 to R17, R16 to R18, R17 to R19, R18 to R20, R19 to R21, R20 to R22, R21 to R23, R22 to R24, R23 to R25, R24 to R26, R25 to R27, R26 to R28, R27 to R29, R2 to R3, R28 to R30, R29 to R31, R30 to R32, R31 to R33, R32 to R34, R33 to R35, R34 to R36, R35 to R37, R36 to R38, R37 to R39, R38 to R40, R39 to R41, R40 to R42, R41 to R43, R42 to R44, R43 to R45, R44 to R46, R45 to R47, R46 to R48, R47 to R49, R4 to R5, R48 to R50, R49 to R51, R50 to R52, R51 to R53, R52 to R54, R53 to R55, R54 to R56, R55 to R57, R56 to R58, R57 to R59, R58 to R60, R59 to R61, R60 to R62, R61 to R63, R62 to R64, R63 to R65, R64 to R66, R65 to R67, R66 to R68, R67 to R69, R68 to R70, R69 to R71, R70 to R72, R71 to R73, R72 to R74, R73 to R75, R74 to R76, R75 to R77, R76 to R78, R77 to R79, R6 to R8, R78 to R80, R79 to R81, R80 to R82, R81 to R83, R82 to R84, R83 to R85, R84 to R86, R85 to R87, R86 to R88, R87 to R89, R7 to R9, R88 to R90, R89 to R91, R90 to R92, R91 to R93, R92 to R94, R93 to R95, R94 to R96, R95 to R97, R96 to R98
Connections:
- J3 pad 2: GND_CAN -> unconnected-(J3-Pin_2-Pad2)
- R7 pad 2: Net-(U4-FB) -> Net-(R6-Pad1)
Routing:
- net U_MES_8: track 34.3 -> 34.9 mm
- net U_BAT_0: track 31.1 -> 30.5 mm
- net 24V0: vias 1 -> 3
- added copper zone on F.Cu, net Net-(D2-K)

Commit message: 20.04.2025_true
Parts:
- L2: footprint user:CTSFW7050F -> user:CDCSAB0420-6R8M
- moved R6 55.4 mm to (159.3, 83.6), turned to 180 degrees
- moved R7 2.28 mm to (159.3, 85.1), turned to 0 degrees
- moved D2 1.53 mm to (150.6, 90.7), turned to -90 degrees
- moved R2 1.53 mm to (205.4, 95.8)
- moved L2 1.48 mm to (154.9, 89.4), turned to 0 degrees
- renumbered R_bal_1 to Rb1, R_bal_2 to Rb2, R_bal_3 to Rb3, R_bal_4 to Rb4, R_bal_5 to Rb5, R_bal_6 to Rb6, R_bal_7 to Rb7, R_bal_8 to Rb8
Routing:
- net TERMO_0: track 96.9 -> 104.2 mm
- net Net-(D2-K): track 9.09 -> 2.33 mm, vias 1 -> 2
- net MPL_TEMP_0_3V3: track 39.6 -> 44.1 mm
- net MPL_VOLT_0_3V3: track 41.5 -> 45.3 mm
- net MPL_VOLT_2_3V3: track 20.9 -> 23.9 mm
- net CAN0-: track 12.9 -> 15.0 mm
- net MPL_VOLT_1_3V3: track 21.3 -> 23.4 mm
- net U_BAT_8: track 52.6 -> 50.6 mm
- net MPL_TEMP_1_3V3: track 16.2 -> 18.1 mm
- net BOOT0: track 0.00 -> 1.82 mm, vias 0 -> 1
- net U_BAT_0: track 30.5 -> 32.3 mm
- net CAN0+: track 26.5 -> 28.2 mm
- net CAN1_STM32_TX: track 114.1 -> 115.6 mm, vias 5 -> 4
- net Net-(R6-Pad1): track 0.00 -> 1.46 mm
- net GND: track 30.9 -> 32.2 mm, vias 29 -> 31
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
Commit message: fix hcpl 21.05.2025
Parts:
- L2: value 6.8 -> 6.8u
- R15, R17, R27, R30, R53, R56: value 500 -> 180
Changed lines of the file:
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@@
 			)
 		)
-		(property "Value" "500"
+		(property "Value" "180"
 			(at 0 1.43 0)
 			(layer "F.Fab")
@@
 			)
 		)
-		(property "Value" "500"
+		(property "Value" "180"
 			(at 0 1.43 90)
 			(layer "F.Fab")
@@
 			)
 		)
-		(property "Value" "500"
+		(property "Value" "180"
 			(at 0 1.43 0)
 			(layer "F.Fab")
@@
 			)
 		)
-		(property "Value" "500"
+		(property "Value" "180"
 			(at 0 1.43 0)
 			(layer "F.Fab")
@@
 			)
 		)
-		(property "Value" "500"
+		(property "Value" "180"
 			(at 0 1.43 0)
 			(layer "F.Fab")
@@
 			)
 		)
-		(property "Value" "500"
+		(property "Value" "180"
 			(at 0 1.43 90)
 			(layer "F.Fab")
@@
 			)
 		)
-		(property "Value" "6.8"
+		(property "Value" "6.8u"
 			(at -0.15 -4.71 180)
 			(unlocked yes)
