File: KiCad/BMS/balance.kicad_sch (KiCad schematic)
At the start: 137 parts, among them Q1 PNP, Q10 NMOS, Q11 PNP, Q12 BSS138, Q13 NMOS, Q14 PNP, Q15 NMOS, Q16 PNP, Q17 NMOS, Q2 NMOS, Q3 PNP, Q4 NMOS, Q5 PNP, Q6 NMOS, Q7 PNP, Q8 NMOS, Q9 PNP, U10 TL431, U11 B0505MT, U12 MCP3201, U13 TL431, U14 HCPL-0630, U15 TL431, U16 HCPL-0600, U17 TL431, U18 HCPL-0600, U19 TL431, U20 TL431, U5 HCPL-0630, U6 TL431, U7 74HC4051, U8 HCPL-0630, U9 TL431

Commit message: 14.03.2025
Parts:
- removed D10, D11, D12, D3, D4, D5, D8, D9: LED_B, LED_SMD:LED_1206_3216Metric, symbol LED:IR26-21C_L110_TR8
- removed R19, R30, R41, R50, R64, R74, R8, R85: 180, Resistor_SMD:R_0603_1608Metric, symbol Device:R
- removed U10, U13, U15, U17, U19, U20, U6, U9: TL431, Package_SO:SOIC-8_3.9x4.9mm_P1.27mm, symbol Reference_Voltage:TL431D
- added U10, U13, U15, U17, U19, U20, U5, U8: TL432DBZ, Package_TO_SOT_SMD:SOT-23, symbol Reference_Voltage:TL432DBZ
- R_bal_1, R_bal_2, R_bal_3, R_bal_4, R_bal_5, R_bal_6, R_bal_7, R_bal_8: footprint Resistor_SMD:R_0603_1608Metric -> Resistor_SMD:R_1206_3216Metric
- renumbered R11 to R10, R12 to R11, R14 to R12, R15 to R13, R10 to R14, R13 to R15, R24 to R23, R25 to R24, R23 to R25, R27 to R26, R28 to R27, R26 to R28, R37 to R36, R38 to R37, R36 to R38, R40 to R39, R39 to R41, R52 to R51, R51 to R52, R54 to R53, R55 to R54, R53 to R55, R57 to R56, R56 to R57, R61 to R62, R62 to R63, R63 to R64, R69 to R68, R70 to R69, R68 to R70, U5 to U6, U8 to U9
Connections:
- net GND_ADC: now also U20.3 (A)
- net U_BAT_1: now also U19.3 (A)
- net at Q8.3 (S), Q9.3 (E), R47.1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: now also U13.3 (A)
- net at R87.1, R88.1, R89.2: now also U20.1 (REF)
- net at R33.1, R35.1, R36.2: now also U10.1 (REF)
- net at Q13.3 (S), Q14.3 (E), R71.1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: now also U17.3 (A)
- net at R77.1: now also U19.2 (K)
- net at R78.1, R80.1, R82.2: now also U19.1 (REF)
- net at R67.1, R69.1, R71.2: now also U17.1 (REF)
- net at Q4.3 (S), Q5.3 (E), R26.1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: now also U8.3 (A)
- net at Q2.3 (S), Q3.3 (E), R16.1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: now also U5.3 (A)
- net at Q10.3 (S), Q11.3 (E), R58.1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: now also U15.3 (A)
- net at R54.1, R56.1, R58.2: now also U15.1 (REF)
- net at Q6.3 (S), Q7.3 (E), R36.1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: now also U10.3 (A)
- net at R22.1, R24.1, R26.2: now also U8.1 (REF)
- net at R21.1: now also U8.2 (K)
- net at R86.1: now also U20.2 (K)
- net at R32.1: now also U10.2 (K)
- net at R11.1, R13.1, R16.2: now also U5.1 (REF)
- net at R44.1, R46.1, R47.2: now also U13.1 (REF)
- net at R43.1: now also U13.2 (K)
- net at R66.1: now also U17.2 (K)
- net at R10.1: now also U5.2 (K)
- net at R53.1: now also U15.2 (K)
Other:
- moved on the sheet: R56

Commit message: 18.03.2025
Parts:
- U10, U13, U15, U17, U19, U20, U5, U8: value TL432DBZ -> TL431A
Changed lines of the file:
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@@
 			)
 		)
-		(property "Value" "TL432DBZ"
+		(property "Value" "TL431A"
 			(at 226.06 307.34 90)
 			(effects
@@
 			)
 		)
-		(property "Value" "TL432DBZ"
+		(property "Value" "TL431A"
 			(at 226.06 139.7 90)
 			(effects
@@
 			)
 		)
-		(property "Value" "TL432DBZ"
+		(property "Value" "TL431A"
 			(at 226.06 349.25 90)
 			(effects
@@
 			)
 		)
-		(property "Value" "TL432DBZ"
+		(property "Value" "TL431A"
 			(at 226.06 97.79 90)
 			(effects
@@
 			)
 		)
-		(property "Value" "TL432DBZ"
+		(property "Value" "TL431A"
 			(at 226.06 181.61 90)
 			(effects
@@
 			)
 		)
-		(property "Value" "TL432DBZ"
+		(property "Value" "TL431A"
 			(at 226.06 265.43 90)
 			(effects
@@
 			)
 		)
-		(property "Value" "TL432DBZ"
+		(property "Value" "TL431A"
 			(at 226.06 59.69 90)
 			(effects
@@
 			)
 		)
-		(property "Value" "TL432DBZ"
+		(property "Value" "TL431A"
 			(at 226.06 223.52 90)
 			(effects

Commit message: 22.03.2025
Parts:
- added J5: 430451000, Connector_Molex:Molex_Micro-Fit_3.0_43045-1000_2x05_P3.00mm_Horizontal, symbol user_lib:430451200
Connections:
- net 5V_ADC: no longer R76.2, U18.6 (VO), U18.8 (VCC)
- net GND_ADC: now also J5.10
- net SPI1_SCK_ADC: no longer U18.5 (GND)
- net U_BAT_1: now also J5.8
- net U_BAT_2: now also J5.7
- net U_BAT_3: now also J5.6
- net U_BAT_4: now also J5.5
- net U_BAT_5: now also J5.4
- net U_BAT_6: now also J5.3
- net U_BAT_7: now also J5.2
- net U_BAT_8: now also J5.1
- net at R76.1: no longer U18.7 (EN)
- no-connect marks 0 -> 1
Other:
- note removed: "ADC (VOLTAGE)"
- note removed: "GALVANIC ISOLATION for ADC"
- note removed: "HIGH SPEED OPTOCOUPLERS for SPI"
- note removed: "MULTIPLEXOR LEVEL CONVERTER"
- note removed: "OVERVOLTAGE PROTECTION for ADC (VOLTAGE)"
- note removed: "PASSIVE BALANCING CIRCUIT"
- moved on the sheet: Q12, Q17, R52, R55, R62, R63, R64, R70, R76, R81, R_bal_1, R_bal_2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

Commit message: 23.03.2025
Parts:
- R81: value 500 -> 180
Connections:
- net SPI1_SCK_ADC is gone; now on net 5V_ADC: U12.7 (CLK)
- net 3V3: now also Q12.1 (G)
- net 5V0: no longer Q12.1 (G)
- net 5V_ADC: now also R76.1, U18.8 (VCC)
- net GND: no longer U14.5 (GND)
- net GND_ADC: now also U14.5 (GND), U18.5 (GND)
- net SPI1_MISO: now also Q12.2 (S); no longer Q12.3 (D)
- net at R63.1, U16.6 (VO): now also Q12.3 (D); no longer Q12.2 (S)
- net at R76.2: now also U18.7 (EN)
Other:
- moved on the sheet: Q12, R76

Commit message: 25.03.2025
Parts:
- added R10, R21, R32, R43: 3m, Resistor_SMD:R_0603_1608Metric, symbol Device:R
- added R7: 1m, Resistor_SMD:R_0603_1608Metric, symbol Device:R
- R20: value 6m -> 3m
- R31: value 5m -> 2m
- R41: renamed from R42; value 4m -> 1m
- R9: value 7m -> 3m
- renumbered D6 to D3, D7 to D4, R10 to R11, R11 to R12, R12 to R15, R15 to R16, R16 to R17, R17 to R18, R18 to R19, R21 to R22, R22 to R23, R23 to R24, R24 to R25, R25 to R26, R26 to R27, R27 to R28, R28 to R29, R29 to R30, R32 to R33, R33 to R34, R34 to R35, R35 to R36, R36 to R37, R37 to R38, R38 to R39, R39 to R40, R41 to R42, R43 to R44, R44 to R45, R45 to R46, R46 to R47, R47 to R48, R48 to R49, R51 to R50, R49 to R51, R57 to R52, R52 to R53, R53 to R54, R54 to R55, R55 to R56, R56 to R57, R65 to R60, R60 to R61, R68 to R65, R69 to R68, R70 to R69, R71 to R70, R72 to R71, R75 to R72, R79 to R74, R77 to R75, R78 to R76, R76 to R77, R80 to R78, R81 to R79, R7 to R8, R82 to R80, R83 to R81, R84 to R82, R86 to R83, R87 to R84, R88 to R85, R89 to R86, R90 to R87, U12 to U11, U11 to U12
Connections:
- net 5V_ADC: no longer U11.7 (CLK)
- net GND_ADC: now also J5.5
- net U_BAT_1: now also J5.9, U7.1 (A4); no longer J5.8, U7.4 (A7)
- net U_BAT_2: now also J5.4, Q13.3 (S), Q14.3 (E), R70.1, R71.1, R72.2, R73.2, R76.2, R_bal_7.2, U17.3 (A); no longer J5.7, R72.1, R74.2, U7.2 (A6)
- net U_BAT_3: now also J5.8, Q10.3 (S), Q11.3 (E), R58.1, R59.1, R60.2, R61.2, R67.2, R_bal_6.2, U15.3 (A); no longer J5.6, R60.1, R65.2, U7.5 (A5)
- net U_BAT_4: now also J5.3, Q8.3 (S), Q9.3 (E), R48.1, R49.1, R50.2, R51.2, R55.2, R_bal_5.2, U13.3 (A); no longer J5.5, R50.1, R52.2, U7.1 (A4)
- net U_BAT_5: now also J5.7, Q6.3 (S), Q7.3 (E), R37.1, R38.1, R40.2, R41.2, R45.2, R_bal_4.2, U10.3 (A); no longer J5.4, R41.1, R46.2, U7.12 (A3)
- net U_BAT_6: now also J5.2, Q4.3 (S), Q5.3 (E), R27.1, R28.1, R30.2, R31.2, R34.2, R_bal_3.2, U8.3 (A); no longer J5.3, R31.1, R35.2, U7.15 (A2)
- net U_BAT_7: now also J5.6, Q2.3 (S), Q3.3 (E), R17.1, R18.1, R19.2, R20.2, R23.2, R_bal_2.2, U5.3 (A); no longer J5.2, R20.1, R24.2, U7.14 (A1)
- net U_BAT_8: now also Q1.3 (E), R12.2, R8.2, R_bal_1.2, R7.1; no longer R15.2, R9.1, U7.13 (A0)
- net SPI1_SCK_ADC: now reaches U18.6 (VO)
- net SPI1_SCK_ADC: now also U11.7 (CLK)
- new net: R31.1, R32.1
- new net: R41.1, R43.1
- new net: R7.2, R9.2
- new net: R20.1, R21.1
- new net: R10.1, R9.1
- new net U_MES_2: R72.1, R74.2, U7.2 (A6)
- new net U_MES_3: R60.1, R65.2, U7.4 (A7)
- new net U_MES_4: R50.1, R52.2, U7.5 (A5)
- new net U_MES_5: R43.2, R46.2, U7.12 (A3)
- new net U_MES_6: R32.2, R35.2, U7.13 (A0)
- new net U_MES_7: R21.2, R24.2, U7.14 (A1)
- new net U_MES_8: R10.2, R15.2, U7.15 (A2)
- no-connect marks 1 -> 0
Other:
- moved on the sheet: J5, R15, R24, R35, R41, R46, R50, R52, R60, R65, R72, R74

Commit message: 27.03.2025
Connections:
- net 5V is gone; now on net 5V0: C23.1, U12.13 (Vin), U12.14 (Vin)
Changed lines of the file:
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@@
 	(text_box "MULTIPLEXOR LEVEL CONVERTER "
 		(exclude_from_sim no)
-		(at -254 -205.74 0)
+		(at 17.78 30.48 0)
 		(size 171.45 99.06)
 		(margins 0.9525 0.9525 0.9525 0.9525)
@@
 			)
 		)
-		(property "Value" "5V"
+		(property "Value" "5V0"
 			(at 162.56 139.7 0)
 			(effects
@@
 			)
 		)
-		(property "Value" "5V"
+		(property "Value" "5V0"
 			(at 135.89 147.32 0)
 			(effects

Commit message: 30.03.2025
Parts:
- removed R42: R, Resistor_SMD:R_0603_1608Metric, symbol Device:R
- D3, D4: value BZX384xxxx -> BZX384-C4V7
Connections:
- net 5V_ADC: now also D3.1 (K)
- net GND_ADC: now also D4.2 (A)
- net U_MEASURE: no longer U11.2 (IN+)
- net U_MEASURE_CLR: now reaches D4.1 (K)
- net U_MEASURE_CLR: now also D3.2 (A), R39.1, U11.2 (IN+)
Other:
- moved on the sheet: D3, D4, R39, U11

Commit message: rough routing is complete (04.04.2025)
Parts:
- renumbered C23 to C25, C24 to C26, J5 to J6, R43 to R42, R44 to R43, R45 to R44, R46 to R45, R47 to R46, R48 to R47, R49 to R48, R50 to R49, R51 to R50, R52 to R51, R53 to R52, R54 to R53, R55 to R54, R56 to R55, R57 to R56, R58 to R57, R59 to R58, R60 to R59, R61 to R60, R62 to R61, R63 to R62, R64 to R63, R65 to R64, R66 to R65, R67 to R66, R68 to R67, R69 to R68, R70 to R69, R71 to R70, R72 to R71, R73 to R72, R74 to R73, R75 to R74, R76 to R75, R77 to R76, R78 to R77, R79 to R78, R80 to R79, R81 to R80, R82 to R81, R83 to R82, R84 to R83, R85 to R84, R86 to R85, R87 to R86, U9 to U10, U10 to U11, U11 to U12, U12 to U13, U13 to U14, U14 to U15, U15 to U16, U16 to U17, U17 to U18, U18 to U19, U19 to U20, U20 to U21, U5 to U6, U6 to U7, U7 to U8, U8 to U9
