File: KiCad/BMS/balance.kicad_sch (KiCad schematic)
At the start: 126 parts, among them J6 430451000, Q1 PNP, Q10 NMOS, Q11 PNP, Q12 BSS138, Q13 NMOS, Q14 PNP, Q15 NMOS, Q16 PNP, Q17 NMOS, Q2 NMOS, Q3 PNP, Q4 NMOS, Q5 PNP, Q6 NMOS, Q7 PNP, Q8 NMOS, Q9 PNP, U10 HCPL-0630, U11 TL431A, U12 MCP3201, U13 B0505MT, U14 TL431A, U15 HCPL-0630, U16 TL431A, U17 HCPL-0600, U18 TL431A, U19 HCPL-0600, U20 TL431A, U21 TL431A, U6 TL431A, U7 HCPL-0630, U8 74HC4051, U9 TL431A

Commit message: 08.04.2025
Parts:
- renumbered R11 to R10, R12 to R11, R13 to R12, R14 to R13, R15 to R14, R16 to R15, R17 to R16, R18 to R17, R19 to R18, R20 to R19, R21 to R20, R22 to R21, R23 to R22, R24 to R23, R25 to R24, R26 to R25, R27 to R26, R28 to R27, R29 to R28, R30 to R29, R31 to R30, R32 to R31, R33 to R32, R34 to R33, R35 to R34, R36 to R35, R37 to R36, R38 to R37, R39 to R38, R40 to R39, R41 to R40, R42 to R41, R43 to R42, R44 to R43, R45 to R44, R46 to R45, R47 to R46, R48 to R47, R49 to R48, R50 to R49, R51 to R50, R52 to R51, R53 to R52, R54 to R53, R55 to R54, R56 to R55, R57 to R56, R58 to R57, R59 to R58, R60 to R59, R7 to R6, R61 to R60, R62 to R61, R63 to R62, R64 to R63, R65 to R64, R66 to R65, R67 to R66, R68 to R67, R69 to R68, R70 to R69, R8 to R7, R71 to R70, R72 to R71, R73 to R72, R74 to R73, R75 to R74, R76 to R75, R77 to R76, R78 to R77, R79 to R78, R80 to R79, R9 to R8, R81 to R80, R82 to R81, R83 to R82, R84 to R83, R85 to R84, R86 to R85, R10 to R9
Connections:
- net 5V0: no longer U15.8 (VCC)
- net 5V_ADC: now also U15.8 (VCC)

Commit message: 19.04.2025
Parts:
- renumbered R8 to R10, R9 to R11, R10 to R12, R11 to R13, R12 to R14, R13 to R15, R14 to R16, R15 to R17, R16 to R18, R17 to R19, R18 to R20, R19 to R21, R20 to R22, R21 to R23, R22 to R24, R23 to R25, R24 to R26, R25 to R27, R26 to R28, R27 to R29, R28 to R30, R29 to R31, R30 to R32, R31 to R33, R32 to R34, R33 to R35, R34 to R36, R35 to R37, R36 to R38, R37 to R39, R38 to R40, R39 to R41, R40 to R42, R41 to R43, R42 to R44, R43 to R45, R44 to R46, R45 to R47, R46 to R48, R47 to R49, R48 to R50, R49 to R51, R50 to R52, R51 to R53, R52 to R54, R53 to R55, R54 to R56, R55 to R57, R56 to R58, R57 to R59, R58 to R60, R59 to R61, R60 to R62, R61 to R63, R62 to R64, R63 to R65, R64 to R66, R65 to R67, R66 to R68, R67 to R69, R68 to R70, R69 to R71, R70 to R72, R71 to R73, R72 to R74, R73 to R75, R74 to R76, R75 to R77, R76 to R78, R77 to R79, R6 to R8, R78 to R80, R79 to R81, R80 to R82, R81 to R83, R82 to R84, R83 to R85, R84 to R86, R85 to R87, R7 to R9

Commit message: 20.04.2025_true
Parts:
- renumbered R_bal_1 to Rb1, R_bal_2 to Rb2, R_bal_3 to Rb3, R_bal_4 to Rb4, R_bal_5 to Rb5, R_bal_6 to Rb6, R_bal_7 to Rb7, R_bal_8 to Rb8
Changed lines of the file:
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@@
 		(on_board yes)
 		(dnp no)
-		(property "Reference" "R_bal_3"
-			(at 262.636 132.08 90)
+		(property "Reference" "Rb3"
+			(at 262.89 130.175 90)
 			(effects
 				(font
@@
 			(project "BMS"
 				(path "/d2402062-308b-4eb4-ada9-28eaf3edc216/0012aeb1-9a62-4ce2-b968-388281bbc3b6"
-					(reference "R_bal_3")
+					(reference "Rb3")
 					(unit 1)
 				)
@@
 		(on_board yes)
 		(dnp no)
-		(property "Reference" "R_bal_5"
-			(at 262.636 215.9 90)
+		(property "Reference" "Rb5"
+			(at 262.89 213.995 90)
 			(effects
 				(font
@@
 			(project "BMS"
 				(path "/d2402062-308b-4eb4-ada9-28eaf3edc216/0012aeb1-9a62-4ce2-b968-388281bbc3b6"
-					(reference "R_bal_5")
+					(reference "Rb5")
 					(unit 1)
 				)
@@
 		(on_board yes)
 		(dnp no)
-		(property "Reference" "R_bal_6"
-			(at 262.636 257.81 90)
+		(property "Reference" "Rb6"
+			(at 262.89 255.905 90)
 			(effects
 				(font
@@
 			(project "BMS"
 				(path "/d2402062-308b-4eb4-ada9-28eaf3edc216/0012aeb1-9a62-4ce2-b968-388281bbc3b6"
-					(reference "R_bal_6")
+					(reference "Rb6")
 					(unit 1)
 				)
@@
 		(on_board yes)
 		(dnp no)
-		(property "Reference" "R_bal_1"
-			(at 262.636 52.07 90)
+		(property "Reference" "Rb1"
+			(at 262.89 50.165 90)
 			(effects
 				(font
@@
 			(project "BMS"
 				(path "/d2402062-308b-4eb4-ada9-28eaf3edc216/0012aeb1-9a62-4ce2-b968-388281bbc3b6"
-					(reference "R_bal_1")
+					(reference "Rb1")
 					(unit 1)
 				)
@@
 		(on_board yes)
 		(dnp no)
-		(property "Reference" "R_bal_8"
-			(at 262.636 341.63 90)
+		(property "Reference" "Rb8"
+			(at 262.89 339.725 90)
 			(effects
 				(font
@@
 			(project "BMS"
 				(path "/d2402062-308b-4eb4-ada9-28eaf3edc216/0012aeb1-9a62-4ce2-b968-388281bbc3b6"
-					(reference "R_bal_8")
+					(reference "Rb8")
 					(unit 1)
 				)
@@
 		(on_board yes)
 		(dnp no)
-		(property "Reference" "R_bal_7"
-			(at 262.636 299.72 90)
+		(property "Reference" "Rb7"
+			(at 262.89 297.815 90)
 			(effects
 				(font
@@
 			(project "BMS"
 				(path "/d2402062-308b-4eb4-ada9-28eaf3edc216/0012aeb1-9a62-4ce2-b968-388281bbc3b6"
-					(reference "R_bal_7")
+					(reference "Rb7")
 					(unit 1)
 				)
@@
 		(on_board yes)
 		(dnp no)
-		(property "Reference" "R_bal_2"
-			(at 262.636 90.17 90)
+		(property "Reference" "Rb2"
+			(at 262.89 88.265 90)
 			(effects
 				(font
@@
 			(project "BMS"
 				(path "/d2402062-308b-4eb4-ada9-28eaf3edc216/0012aeb1-9a62-4ce2-b968-388281bbc3b6"
-					(reference "R_bal_2")
+					(reference "Rb2")
 					(unit 1)
 				)
@@
 		(on_board yes)
 		(dnp no)
-		(property "Reference" "R_bal_4"
-			(at 262.636 173.99 90)
+		(property "Reference" "Rb4"
+			(at 262.89 172.085 90)
 			(effects
 				(font
@@
 			(project "BMS"
 				(path "/d2402062-308b-4eb4-ada9-28eaf3edc216/0012aeb1-9a62-4ce2-b968-388281bbc3b6"
-					(reference "R_bal_4")
+					(reference "Rb4")
 					(unit 1)
 				)

Commit message: fix hcpl 21.05.2025
Parts:
- R15, R17, R27, R30, R53, R56: value 500 -> 180
Changed lines of the file:
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@@
 			)
 		)
-		(property "Value" "500"
+		(property "Value" "180"
 			(at 66.04 64.77 90)
 			(effects
@@
 			)
 		)
-		(property "Value" "500"
+		(property "Value" "180"
 			(at 66.04 102.87 90)
 			(effects
@@
 			)
 		)
-		(property "Value" "500"
+		(property "Value" "180"
 			(at 59.69 218.44 90)
 			(effects
@@
 			)
 		)
-		(property "Value" "500"
+		(property "Value" "180"
 			(at 66.04 59.69 90)
 			(effects
@@
 			)
 		)
-		(property "Value" "500"
+		(property "Value" "180"
 			(at 66.04 107.95 90)
 			(effects
@@
 			)
 		)
-		(property "Value" "500"
+		(property "Value" "180"
 			(at 59.69 213.36 90)
 			(effects

Commit message: 22.05.2025
Parts:
- R69: value 500 -> 470
Changed lines of the file:
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@@
 			)
 		)
-		(property "Value" "500"
+		(property "Value" "470"
 			(at 100.33 265.43 90)
 			(effects
