File: KiCad/BMS/_autosave-BMS.kicad_pcb (KiCad board)
At the start: 4 copper layers, 129.3 x 93.6 mm, 196 parts, among them J1 PLS-6, J2 BH1,27-10-G, J3 430450400, J4 Conn_01x03, J5 430450400, J6 430451000, J7 430450800, J8 430450800, Q1 PNP, Q10 NMOS, Q11 PNP, Q12 BSS138, Q13 NMOS, Q14 PNP, Q15 NMOS, Q16 PNP, Q17 NMOS, Q2 NMOS, Q3 PNP, Q4 NMOS, Q5 PNP, Q6 NMOS, Q7 PNP, Q8 NMOS, Q9 PNP, SW1 B3F1060, U1 STM32F405RGTx, U10 HCPL-0630, U11 TL431A, U12 MCP3201, U13 B0505MT, U14 TL431A, U15 HCPL-0630, U16 TL431A, U17 HCPL-0600, U18 TL431A, U19 HCPL-0600, U2 ISO1050DUB, U20 TL431A, U21 TL431A, U22 MCP3201, U23 74HC4051, U24 HCPL-0630, U3 B0505MT, U4 ST1S14PHR, U5 LDL1117S33R, U6 TL431A, U7 HCPL-0630, U8 74HC4051, U9 TL431A, Y1 Crystal KSE-7U08000MAB143ZA3

Commit message: pupupu
Routing:
- net T_MEASURE_CLR: track 33.5 -> 34.9 mm
- net U_MEASURE_CLR: track 15.9 -> 16.9 mm
- net U_BAT_0: vias 14 -> 16
- added copper zone on In1.Cu, net 5V0
- added copper zone on In2.Cu, net U_BAT_0
