File: KiCad/BMS/termistors.kicad_sch (KiCad schematic)
At the start: 18 parts, among them J4 430451200, U21 74HC4051, U22 MCP3201, U23 HCPL-0630

Commit message: 14.03.2025
Parts:
- renumbered J4 to J5
Changed lines of the file:
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@@
 		(dnp no)
 		(fields_autoplaced yes)
-		(property "Reference" "J4"
+		(property "Reference" "J5"
 			(at 107.95 95.25 0)
 			(effects
@@
 			(project "BMS"
 				(path "/d2402062-308b-4eb4-ada9-28eaf3edc216/3a9bc664-ddd4-401c-aeae-409c2a66a647"
-					(reference "J4")
+					(reference "J5")
 					(unit 1)
 				)

Commit message: 22.03.2025
Parts:
- removed J5: 430451200, Connector_Molex:Molex_Micro-Fit_3.0_43045-1200_2x06_P3.00mm_Horizontal, symbol user_lib:430451200
- added J8, J9: 430450800, Connector_Molex:Molex_Micro-Fit_3.0_43045-0800_2x04_P3.00mm_Horizontal, symbol Connector_Generic:Conn_02x04_Counter_Clockwise
Connections:
- net TERMO_0_OUT: now also J8.1 (Pin_1)
- net TERMO_1_OUT: now also J8.2 (Pin_2)
- net TERMO_2_OUT: now also J8.3 (Pin_3)
- net TERMO_3_OUT: now also J8.4 (Pin_4)
- net TERMO_4_OUT: now also J9.1 (Pin_1)
- net TERMO_5_OUT: now also J9.2 (Pin_2)
- net TERMO_6_OUT: now also J9.3 (Pin_3)
- net TERMO_7_OUT: now also J9.4 (Pin_4)
- net U_BAT_0: now also J8.5 (Pin_5), J8.6 (Pin_6), J8.7 (Pin_7), J8.8 (Pin_8), J9.5 (Pin_5), J9.6 (Pin_6), J9.7 (Pin_7), J9.8 (Pin_8)
- no-connect marks 3 -> 0
Other:
- note removed: "ADC (TEMPERATURE)"
- note removed: "OVERVOLTAGE PROTECTION for ADC (TEMPERATURE)"
- moved on the sheet: D13, D14, R91, R92, U22

Commit message: 25.03.2025
Parts:
- renumbered D13 to D5, D14 to D6, J8 to J6, J9 to J7, R91 to R88, R92 to R89, R93 to R90, R94 to R91, R95 to R92, R96 to R93, R97 to R94, R98 to R95, R99 to R96, R100 to R97, R101 to R98, R102 to R99
Changed lines of the file:
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@@
 		(on_board yes)
 		(dnp no)
-		(property "Reference" "R99"
+		(property "Reference" "R96"
 			(at 54.61 120.65 90)
 			(effects
@@
 			(project "BMS"
 				(path "/d2402062-308b-4eb4-ada9-28eaf3edc216/3a9bc664-ddd4-401c-aeae-409c2a66a647"
-					(reference "R99")
+					(reference "R96")
 					(unit 1)
 				)
@@
 		(on_board yes)
 		(dnp no)
-		(property "Reference" "D13"
+		(property "Reference" "D5"
 			(at 68.58 52.0701 90)
 			(effects
@@
 			(project "BMS"
 				(path "/d2402062-308b-4eb4-ada9-28eaf3edc216/3a9bc664-ddd4-401c-aeae-409c2a66a647"
-					(reference "D13")
+					(reference "D5")
 					(unit 1)
 				)
@@
 		(on_board yes)
 		(dnp no)
-		(property "Reference" "#PWR059"
+		(property "Reference" "#PWR061"
 			(at 85.09 74.93 0)
 			(effects
@@
 			(project "BMS"
 				(path "/d2402062-308b-4eb4-ada9-28eaf3edc216/3a9bc664-ddd4-401c-aeae-409c2a66a647"
-					(reference "#PWR059")
+					(reference "#PWR061")
 					(unit 1)
 				)
@@
 		(dnp no)
 		(fields_autoplaced yes)
-		(property "Reference" "#PWR063"
+		(property "Reference" "#PWR064"
 			(at 194.31 105.41 0)
 			(effects
@@
 			(project "BMS"
 				(path "/d2402062-308b-4eb4-ada9-28eaf3edc216/3a9bc664-ddd4-401c-aeae-409c2a66a647"
-					(reference "#PWR063")
+					(reference "#PWR064")
 					(unit 1)
 				)
@@
 		(on_board yes)
 		(dnp no)
-		(property "Reference" "R98"
+		(property "Reference" "R95"
 			(at 220.98 118.11 90)
 			(effects
@@
 			(project "BMS"
 				(path "/d2402062-308b-4eb4-ada9-28eaf3edc216/3a9bc664-ddd4-401c-aeae-409c2a66a647"
-					(reference "R98")
+					(reference "R95")
 					(unit 1)
 				)
@@
 		(on_board yes)
 		(dnp no)
-		(property "Reference" "#PWR064"
+		(property "Reference" "#PWR065"
 			(at 237.49 105.41 0)
 			(effects
@@
 			(project "BMS"
 				(path "/d2402062-308b-4eb4-ada9-28eaf3edc216/3a9bc664-ddd4-401c-aeae-409c2a66a647"
-					(reference "#PWR064")
+					(reference "#PWR065")
 					(unit 1)
 				)
@@
 		(on_board yes)
 		(dnp no)
-		(property "Reference" "J8"
+		(property "Reference" "J6"
 			(at 118.11 100.33 0)
 			(effects
@@
 			(project "BMS"
 				(path "/d2402062-308b-4eb4-ada9-28eaf3edc216/3a9bc664-ddd4-401c-aeae-409c2a66a647"
-					(reference "J8")
+					(reference "J6")
 					(unit 1)
 				)
@@
 		(on_board yes)
 		(dnp no)
-		(property "Reference" "#PWR057"
+		(property "Reference" "#PWR058"
 			(at 218.44 39.37 0)
 			(effects
@@
 			(project "BMS"
 				(path "/d2402062-308b-4eb4-ada9-28eaf3edc216/3a9bc664-ddd4-401c-aeae-409c2a66a647"
-					(reference "#PWR057")
+					(reference "#PWR058")
 					(unit 1)
 				)
@@
 		(on_board yes)
 		(dnp no)
-		(property "Reference" "R92"
+		(property "Reference" "R89"
 			(at 77.47 63.5 90)
 			(effects
@@
 			(project "BMS"
 				(path "/d2402062-308b-4eb4-ada9-28eaf3edc216/3a9bc664-ddd4-401c-aeae-409c2a66a647"
-					(reference "R92")
+					(reference "R89")
 					(unit 1)
 				)
@@
 		(on_board yes)
 		(dnp no)
-		(property "Reference" "R91"
+		(property "Reference" "R88"
 			(at 77.47 43.18 90)
 			(effects
@@
 			(project "BMS"
 				(path "/d2402062-308b-4eb4-ada9-28eaf3edc216/3a9bc664-ddd4-401c-aeae-409c2a66a647"
-					(reference "R91")
+					(reference "R88")
 					(unit 1)
 				)
@@
 		(on_board yes)
 		(dnp no)
-		(property "Reference" "D14"
+		(property "Reference" "D6"
 			(at 68.58 59.6899 90)
 			(effects
@@
 			(project "BMS"
 				(path "/d2402062-308b-4eb4-ada9-28eaf3edc216/3a9bc664-ddd4-401c-aeae-409c2a66a647"
-					(reference "D14")
+					(reference "D6")
 					(unit 1)
 				)
@@
 		(on_board yes)
 		(dnp no)
-		(property "Reference" "R94"
+		(property "Reference" "R91"
 			(at 54.61 105.41 90)
 			(effects
@@
 			(project "BMS"
 				(path "/d2402062-308b-4eb4-ada9-28eaf3edc216/3a9bc664-ddd4-401c-aeae-409c2a66a647"
-					(reference "R94")
+					(reference "R91")
 					(unit 1)
 				)
@@
 		(on_board yes)
 		(dnp no)
-		(property "Reference" "R101"
+		(property "Reference" "R98"
 			(at 54.61 130.81 90)
 			(effects
@@
 			(project "BMS"
 				(path "/d2402062-308b-4eb4-ada9-28eaf3edc216/3a9bc664-ddd4-401c-aeae-409c2a66a647"
-					(reference "R101")
+					(reference "R98")
 					(unit 1)
 				)
@@
 		(on_board yes)
 		(dnp no)
-		(property "Reference" "#PWR058"
+		(property "Reference" "#PWR059"
 			(at 147.32 46.99 0)
 			(effects
@@
 			(project "BMS"
 				(path "/d2402062-308b-4eb4-ada9-28eaf3edc216/3a9bc664-ddd4-401c-aeae-409c2a66a647"
-					(reference "#PWR058")
+					(reference "#PWR059")
 					(unit 1)
 				)
@@
 		(dnp no)
 		(fields_autoplaced yes)
-		(property "Reference" "#PWR061"
+		(property "Reference" "#PWR062"
 			(at 215.9 77.47 0)
 			(effects
@@
 			(project "BMS"
 				(path "/d2402062-308b-4eb4-ada9-28eaf3edc216/3a9bc664-ddd4-401c-aeae-409c2a66a647"
-					(reference "#PWR061")
+					(reference "#PWR062")
 					(unit 1)
 				)
@@
 		(on_board yes)
 		(dnp no)
-		(property "Reference" "R96"
+		(property "Reference" "R93"
 			(at 220.98 113.03 90)
 			(effects
@@
 			(project "BMS"
 				(path "/d2402062-308b-4eb4-ada9-28eaf3edc216/3a9bc664-ddd4-401c-aeae-409c2a66a647"
-					(reference "R96")
+					(reference "R93")
 					(unit 1)
 				)
@@
 		(on_board yes)
 		(dnp no)
-		(property "Reference" "R95"
+		(property "Reference" "R92"
 			(at 54.61 110.49 90)
 			(effects
@@
 			(project "BMS"
 				(path "/d2402062-308b-4eb4-ada9-28eaf3edc216/3a9bc664-ddd4-401c-aeae-409c2a66a647"
-					(reference "R95")
+					(reference "R92")
 					(unit 1)
 				)
@@
 		(on_board yes)
 		(dnp no)
-		(property "Reference" "#PWR065"
+		(property "Reference" "#PWR066"
 			(at 237.49 139.7 0)
 			(effects
@@
 			(project "BMS"
 				(path "/d2402062-308b-4eb4-ada9-28eaf3edc216/3a9bc664-ddd4-401c-aeae-409c2a66a647"
-					(reference "#PWR065")
+					(reference "#PWR066")
 					(unit 1)
 				)
@@
 		(on_board yes)
 		(dnp no)
-		(property "Reference" "R102"
+		(property "Reference" "R99"
 			(at 54.61 135.89 90)
 			(effects
@@
 			(project "BMS"
 				(path "/d2402062-308b-4eb4-ada9-28eaf3edc216/3a9bc664-ddd4-401c-aeae-409c2a66a647"
-					(reference "R102")
+					(reference "R99")
 					(unit 1)
 				)
@@
 		(on_board yes)
 		(dnp no)
-		(property "Reference" "R100"
+		(property "Reference" "R97"
 			(at 54.61 125.73 90)
 			(effects
@@
 			(project "BMS"
 				(path "/d2402062-308b-4eb4-ada9-28eaf3edc216/3a9bc664-ddd4-401c-aeae-409c2a66a647"
-					(reference "R100")
+					(reference "R97")
 					(unit 1)
 				)
@@
 		(on_board yes)
 		(dnp no)
-		(property "Reference" "R93"
+		(property "Reference" "R90"
 			(at 54.61 100.33 90)
 			(effects
@@
 			(project "BMS"
 				(path "/d2402062-308b-4eb4-ada9-28eaf3edc216/3a9bc664-ddd4-401c-aeae-409c2a66a647"
-					(reference "R93")
+					(reference "R90")
 					(unit 1)
 				)
@@
 		(on_board yes)
 		(dnp no)
-		(property "Reference" "R97"
+		(property "Reference" "R94"
 			(at 54.61 115.57 90)
 			(effects
@@
 			(project "BMS"
 				(path "/d2402062-308b-4eb4-ada9-28eaf3edc216/3a9bc664-ddd4-401c-aeae-409c2a66a647"
-					(reference "R97")
+					(reference "R94")
 					(unit 1)
 				)
@@
 		(on_board yes)
 		(dnp no)
-		(property "Reference" "J9"
+		(property "Reference" "J7"
 			(at 118.11 116.84 0)
 			(effects
@@
 			(project "BMS"
 				(path "/d2402062-308b-4eb4-ada9-28eaf3edc216/3a9bc664-ddd4-401c-aeae-409c2a66a647"
-					(reference "J9")
+					(reference "J7")
 					(unit 1)
 				)
@@
 		(on_board yes)
 		(dnp no)
-		(property "Reference" "#PWR062"
+		(property "Reference" "#PWR063"
 			(at 48.26 102.87 0)
 			(effects
@@
 			(project "BMS"
 				(path "/d2402062-308b-4eb4-ada9-28eaf3edc216/3a9bc664-ddd4-401c-aeae-409c2a66a647"
-					(reference "#PWR062")
-					(unit 1)
-				)
+					(reference "#PWR063")
+					(unit 1)
+				)

Commit message: 27.03.2025
Connections:
- net TERMO_0_IN: now also U21.4 (A7)
- net TERMO_0_OUT: no longer U21.4 (A7)
- net TERMO_1_IN: now also U21.2 (A6)
- net TERMO_1_OUT: no longer U21.2 (A6)
- net TERMO_2_IN: now also U21.5 (A5)
- net TERMO_2_OUT: no longer U21.5 (A5)
- net TERMO_3_IN: now also U21.1 (A4)
- net TERMO_3_OUT: no longer U21.1 (A4)
- net TERMO_4_IN: now also U21.12 (A3)
- net TERMO_4_OUT: no longer U21.12 (A3)
- net TERMO_5_IN: now also U21.15 (A2)
- net TERMO_5_OUT: no longer U21.15 (A2)
- net TERMO_6_IN: now also U21.14 (A1)
- net TERMO_6_OUT: no longer U21.14 (A1)
- net TERMO_7_IN: now also U21.13 (A0)
- net TERMO_7_OUT: no longer U21.13 (A0)
Other:
- moved on the sheet: D5, D6, R88, R89, U21, U22

Commit message: 30.03.2025
Parts:
- removed D5, D6: BZX384xxxx, Diode_SMD:D_SOD-323_HandSoldering, symbol Diode:BZX384xxxx
- removed R88, R89: R, Resistor_SMD:R_0603_1608Metric, symbol Device:R
- added D7, D8: BZX384-C4V7, Diode_SMD:D_SOD-323_HandSoldering, symbol Diode:BZX384xxxx
- added R42: R, Resistor_SMD:R_0603_1608Metric, symbol Device:R
Connections:
- net 5V_ADC: now also D8.1 (K)
- net GND_ADC: now also D7.2 (A)
- net T_MEASURE: now also R42.2; no longer U22.2 (IN+)
- new net T_MEASURE_CLR: D7.1 (K), D8.2 (A), R42.1, U22.2 (IN+)
Other:
- moved on the sheet: U22

Commit message: rough routing is complete (04.04.2025)
Parts:
- renumbered D8 to D5, D7 to D6, J6 to J7, J7 to J8, R42 to R87, R90 to R88, R91 to R89, R92 to R90, R93 to R91, R94 to R92, R95 to R93, R96 to R94, R97 to R95, R98 to R96, R99 to R97, U21 to U23, U23 to U24
Connections:
- net TERMO_0_OUT is gone; now on net TERMO_0: J7.1 (Pin_1)
- net TERMO_1_OUT is gone; now on net TERMO_1: J7.2 (Pin_2)
- net TERMO_2_OUT is gone; now on net TERMO_2: J7.3 (Pin_3)
- net TERMO_3_OUT is gone; now on net TERMO_3: J7.4 (Pin_4)
- net TERMO_4_OUT is gone; now on net TERMO_4: J8.1 (Pin_1)
- net TERMO_5_OUT is gone; now on net TERMO_5: J8.2 (Pin_2)
- net TERMO_6_OUT is gone; now on net TERMO_6: J8.3 (Pin_3)
- net TERMO_7_OUT is gone; now on net TERMO_7: J8.4 (Pin_4)
- net TERMO_0_IN renamed TERMO_0
- net TERMO_1_IN renamed TERMO_1
- net TERMO_2_IN renamed TERMO_2
- net TERMO_3_IN renamed TERMO_3
- net TERMO_4_IN renamed TERMO_4
- net TERMO_5_IN renamed TERMO_5
- net TERMO_6_IN renamed TERMO_6
- net TERMO_7_IN renamed TERMO_7

Commit message: 08.04.2025
Parts:
- renumbered R87 to R86, R88 to R87, R89 to R88, R90 to R89, R91 to R90, R92 to R91, R93 to R92, R94 to R93, R95 to R94, R96 to R95, R97 to R96
Changed lines of the file:
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@@
 		(on_board yes)
 		(dnp no)
-		(property "Reference" "R94"
+		(property "Reference" "R93"
 			(at 54.61 120.65 90)
 			(effects
@@
 			(project "BMS"
 				(path "/d2402062-308b-4eb4-ada9-28eaf3edc216/3a9bc664-ddd4-401c-aeae-409c2a66a647"
-					(reference "R94")
+					(reference "R93")
 					(unit 1)
 				)
@@
 		(dnp no)
 		(fields_autoplaced yes)
-		(property "Reference" "#PWR076"
+		(property "Reference" "#PWR075"
 			(at 194.31 105.41 0)
 			(effects
@@
 			(project "BMS"
 				(path "/d2402062-308b-4eb4-ada9-28eaf3edc216/3a9bc664-ddd4-401c-aeae-409c2a66a647"
-					(reference "#PWR076")
+					(reference "#PWR075")
 					(unit 1)
 				)
@@
 		(on_board yes)
 		(dnp no)
-		(property "Reference" "#PWR070"
+		(property "Reference" "#PWR069"
 			(at 182.88 48.26 0)
 			(effects
@@
 			(project "BMS"
 				(path "/d2402062-308b-4eb4-ada9-28eaf3edc216/3a9bc664-ddd4-401c-aeae-409c2a66a647"
-					(reference "#PWR070")
+					(reference "#PWR069")
 					(unit 1)
 				)
@@
 		(on_board yes)
 		(dnp no)
-		(property "Reference" "R93"
+		(property "Reference" "R92"
 			(at 220.98 118.11 90)
 			(effects
@@
 			(project "BMS"
 				(path "/d2402062-308b-4eb4-ada9-28eaf3edc216/3a9bc664-ddd4-401c-aeae-409c2a66a647"
-					(reference "R93")
+					(reference "R92")
 					(unit 1)
 				)
@@
 		(on_board yes)
 		(dnp no)
-		(property "Reference" "#PWR073"
+		(property "Reference" "#PWR072"
 			(at 236.22 71.12 0)
 			(effects
@@
 			(project "BMS"
 				(path "/d2402062-308b-4eb4-ada9-28eaf3edc216/3a9bc664-ddd4-401c-aeae-409c2a66a647"
-					(reference "#PWR073")
+					(reference "#PWR072")
 					(unit 1)
 				)
@@
 		(on_board yes)
 		(dnp no)
-		(property "Reference" "#PWR077"
+		(property "Reference" "#PWR076"
 			(at 237.49 105.41 0)
 			(effects
@@
 			(project "BMS"
 				(path "/d2402062-308b-4eb4-ada9-28eaf3edc216/3a9bc664-ddd4-401c-aeae-409c2a66a647"
-					(reference "#PWR077")
+					(reference "#PWR076")
 					(unit 1)
 				)
@@
 		(on_board yes)
 		(dnp no)
-		(property "Reference" "#PWR071"
+		(property "Reference" "#PWR070"
 			(at 91.44 52.07 0)
 			(effects
@@
 			(project "BMS"
 				(path "/d2402062-308b-4eb4-ada9-28eaf3edc216/3a9bc664-ddd4-401c-aeae-409c2a66a647"
-					(reference "#PWR071")
+					(reference "#PWR070")
 					(unit 1)
 				)
@@
 		(on_board yes)
 		(dnp no)
-		(property "Reference" "R89"
+		(property "Reference" "R88"
 			(at 54.61 105.41 90)
 			(effects
@@
 			(project "BMS"
 				(path "/d2402062-308b-4eb4-ada9-28eaf3edc216/3a9bc664-ddd4-401c-aeae-409c2a66a647"
-					(reference "R89")
+					(reference "R88")
 					(unit 1)
 				)
@@
 		(on_board yes)
 		(dnp no)
-		(property "Reference" "R96"
+		(property "Reference" "R95"
 			(at 54.61 130.81 90)
 			(effects
@@
 			(project "BMS"
 				(path "/d2402062-308b-4eb4-ada9-28eaf3edc216/3a9bc664-ddd4-401c-aeae-409c2a66a647"
-					(reference "R96")
+					(reference "R95")
 					(unit 1)
 				)
@@
 		(on_board yes)
 		(dnp no)
-		(property "Reference" "#PWR069"
+		(property "Reference" "#PWR068"
 			(at 236.22 44.45 0)
 			(effects
@@
 			(project "BMS"
 				(path "/d2402062-308b-4eb4-ada9-28eaf3edc216/3a9bc664-ddd4-401c-aeae-409c2a66a647"
-					(reference "#PWR069")
+					(reference "#PWR068")
 					(unit 1)
 				)
@@
 		(dnp no)
 		(fields_autoplaced yes)
-		(property "Reference" "#PWR074"
+		(property "Reference" "#PWR073"
 			(at 88.9 90.17 0)
 			(effects
@@
 			(project "BMS"
 				(path "/d2402062-308b-4eb4-ada9-28eaf3edc216/3a9bc664-ddd4-401c-aeae-409c2a66a647"
-					(reference "#PWR074")
+					(reference "#PWR073")
 					(unit 1)
 				)
@@
 		(on_board yes)
 		(dnp no)
-		(property "Reference" "R91"
+		(property "Reference" "R90"
 			(at 220.98 113.03 90)
 			(effects
@@
 			(project "BMS"
 				(path "/d2402062-308b-4eb4-ada9-28eaf3edc216/3a9bc664-ddd4-401c-aeae-409c2a66a647"
-					(reference "R91")
+					(reference "R90")
 					(unit 1)
 				)
@@
 		(on_board yes)
 		(dnp no)
-		(property "Reference" "R90"
+		(property "Reference" "R89"
 			(at 54.61 110.49 90)
 			(effects
@@
 			(project "BMS"
 				(path "/d2402062-308b-4eb4-ada9-28eaf3edc216/3a9bc664-ddd4-401c-aeae-409c2a66a647"
-					(reference "R90")
+					(reference "R89")
 					(unit 1)
 				)
@@
 		(on_board yes)
 		(dnp no)
-		(property "Reference" "#PWR078"
+		(property "Reference" "#PWR077"
 			(at 237.49 139.7 0)
 			(effects
@@
 			(project "BMS"
 				(path "/d2402062-308b-4eb4-ada9-28eaf3edc216/3a9bc664-ddd4-401c-aeae-409c2a66a647"
-					(reference "#PWR078")
+					(reference "#PWR077")
 					(unit 1)
 				)
@@
 		(on_board yes)
 		(dnp no)
-		(property "Reference" "R97"
+		(property "Reference" "R96"
 			(at 54.61 135.89 90)
 			(effects
@@
 			(project "BMS"
 				(path "/d2402062-308b-4eb4-ada9-28eaf3edc216/3a9bc664-ddd4-401c-aeae-409c2a66a647"
-					(reference "R97")
+					(reference "R96")
 					(unit 1)
 				)
@@
 		(on_board yes)
 		(dnp no)
-		(property "Reference" "R95"
+		(property "Reference" "R94"
 			(at 54.61 125.73 90)
 			(effects
@@
 			(project "BMS"
 				(path "/d2402062-308b-4eb4-ada9-28eaf3edc216/3a9bc664-ddd4-401c-aeae-409c2a66a647"
-					(reference "R95")
+					(reference "R94")
 					(unit 1)
 				)
@@
 		(on_board yes)
 		(dnp no)
-		(property "Reference" "R87"
+		(property "Reference" "R86"
 			(at 166.37 49.53 90)
 			(effects
@@
 			(project "BMS"
 				(path "/d2402062-308b-4eb4-ada9-28eaf3edc216/3a9bc664-ddd4-401c-aeae-409c2a66a647"
-					(reference "R87")
+					(reference "R86")
 					(unit 1)
 				)
@@
 		(on_board yes)
 		(dnp no)
-		(property "Reference" "R88"
+		(property "Reference" "R87"
 			(at 54.61 100.33 90)
 			(effects
@@
 			(project "BMS"
 				(path "/d2402062-308b-4eb4-ada9-28eaf3edc216/3a9bc664-ddd4-401c-aeae-409c2a66a647"
-					(reference "R88")
+					(reference "R87")
 					(unit 1)
 				)
@@
 		(on_board yes)
 		(dnp no)
-		(property "Reference" "R92"
+		(property "Reference" "R91"
 			(at 54.61 115.57 90)
 			(effects
@@
 			(project "BMS"
 				(path "/d2402062-308b-4eb4-ada9-28eaf3edc216/3a9bc664-ddd4-401c-aeae-409c2a66a647"
-					(reference "R92")
+					(reference "R91")
 					(unit 1)
 				)
@@
 		(on_board yes)
 		(dnp no)
-		(property "Reference" "#PWR075"
+		(property "Reference" "#PWR074"
 			(at 48.26 102.87 0)
 			(effects
@@
 			(project "BMS"
 				(path "/d2402062-308b-4eb4-ada9-28eaf3edc216/3a9bc664-ddd4-401c-aeae-409c2a66a647"
-					(reference "#PWR075")
+					(reference "#PWR074")
 					(unit 1)
 				)
@@
 		(on_board yes)
 		(dnp no)
-		(property "Reference" "#PWR072"
+		(property "Reference" "#PWR071"
 			(at 172.72 66.04 0)
 			(effects
@@
 			(project "BMS"
 				(path "/d2402062-308b-4eb4-ada9-28eaf3edc216/3a9bc664-ddd4-401c-aeae-409c2a66a647"
-					(reference "#PWR072")
-					(unit 1)
-				)
+					(reference "#PWR071")
+					(unit 1)
+				)

Commit message: 18.04.2025_final
Parts:
- renumbered R93 to R87, R94 to R88, R95 to R89, R96 to R91, R87 to R93, R88 to R94, R91 to R95, R89 to R96
Connections:
- net TERMO_0: now also R88.2, U23.15 (A2); no longer R93.2, U23.4 (A7)
- net TERMO_1: now also R89.2, U23.14 (A1); no longer R94.2, U23.2 (A6)
- net TERMO_2: now also R87.2, U23.12 (A3); no longer R96.2, U23.5 (A5)
- net TERMO_3: now also R91.2, U23.13 (A0); no longer R95.2, U23.1 (A4)
- net TERMO_4: now also R93.2, U23.4 (A7); no longer R87.2, U23.12 (A3)
- net TERMO_5: now also R94.2, U23.2 (A6); no longer R88.2, U23.15 (A2)
- net TERMO_6: now also R95.2, U23.1 (A4); no longer R89.2, U23.14 (A1)
- net TERMO_7: now also R96.2, U23.5 (A5); no longer R91.2, U23.13 (A0)
Other:
- moved on the sheet: R87, R88, R89, R91, R93, R94, R95, R96
