File: KiCad/BMS/BMS.kicad_sch (KiCad schematic)
At the start: 21 parts, among them J1 PLS-6, J2 BH1,27-10-G, SW1 B3F1060, SW2 MSS-12D16, U1 STM32F405RGTx, Y1 Crystal

Commit message: 14.03.2025
Parts:
- renumbered C9 to C10, C10 to C9
Changed lines of the file:
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@@
 		(dnp no)
 		(fields_autoplaced yes)
-		(property "Reference" "C10"
+		(property "Reference" "C9"
 			(at 222.885 31.7499 0)
 			(effects
@@
 			(project "BMS"
 				(path "/d2402062-308b-4eb4-ada9-28eaf3edc216"
-					(reference "C10")
+					(reference "C9")
 					(unit 1)
 				)
@@
 		(dnp no)
 		(fields_autoplaced yes)
-		(property "Reference" "C9"
+		(property "Reference" "C10"
 			(at 198.12 33.0199 0)
 			(effects
@@
 			(project "BMS"
 				(path "/d2402062-308b-4eb4-ada9-28eaf3edc216"
-					(reference "C9")
+					(reference "C10")
 					(unit 1)
 				)

Commit message: 22.03.2025
Connections:
- net CAN1_STM32_RX: now also U1.44 (PA11); no longer U1.45 (PA12)
- net CAN1_STM32_TX: now also U1.45 (PA12); no longer U1.44 (PA11)
- net NRST: no longer R2.1
- net BOOT0: now reaches U1.60 (BOOT0)
- net BOOT0: now also R2.1
Other:
- added sheet FIXING (fixing.kicad_sch)
- note removed: "BOOT0"
- note removed: "OSC"
- note removed: "POWER SUPPLY"
- note removed: "RESET"
- note removed: "SWD Debug connectors"
- note removed: "VCAP"
- moved on the sheet: C1, C10, C11, C12, R2, SW2

Commit message: 25.03.2025
Parts:
- Y1: value Crystal -> Crystal KSE-7U08000MAB143ZA3
- renumbered C9 to C10, C10 to C9
Changed lines of the file:
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@@
 			)
 		)
-		(property "Value" "Crystal"
+		(property "Value" "Crystal KSE-7U08000MAB143ZA3"
 			(at 207.01 19.304 0)
 			(effects
@@
 		(dnp no)
 		(fields_autoplaced yes)
-		(property "Reference" "#PWR04"
+		(property "Reference" "#PWR06"
 			(at 259.08 45.72 0)
 			(effects
@@
 			(project "BMS"
 				(path "/d2402062-308b-4eb4-ada9-28eaf3edc216"
-					(reference "#PWR04")
+					(reference "#PWR06")
 					(unit 1)
 				)
@@
 		(dnp no)
 		(fields_autoplaced yes)
-		(property "Reference" "#PWR06"
+		(property "Reference" "#PWR05"
 			(at 160.02 44.45 0)
 			(effects
@@
 			(project "BMS"
 				(path "/d2402062-308b-4eb4-ada9-28eaf3edc216"
-					(reference "#PWR06")
+					(reference "#PWR05")
 					(unit 1)
 				)
@@
 		(dnp no)
 		(fields_autoplaced yes)
-		(property "Reference" "C9"
+		(property "Reference" "C10"
 			(at 222.885 31.7499 0)
 			(effects
@@
 			(project "BMS"
 				(path "/d2402062-308b-4eb4-ada9-28eaf3edc216"
-					(reference "C9")
+					(reference "C10")
 					(unit 1)
 				)
@@
 		(dnp no)
 		(fields_autoplaced yes)
-		(property "Reference" "#PWR05"
+		(property "Reference" "#PWR04"
 			(at 106.68 44.45 0)
 			(effects
@@
 			(project "BMS"
 				(path "/d2402062-308b-4eb4-ada9-28eaf3edc216"
-					(reference "#PWR05")
+					(reference "#PWR04")
 					(unit 1)
 				)
@@
 		(dnp no)
 		(fields_autoplaced yes)
-		(property "Reference" "C10"
+		(property "Reference" "C9"
 			(at 198.12 31.7499 0)
 			(effects
@@
 			(project "BMS"
 				(path "/d2402062-308b-4eb4-ada9-28eaf3edc216"
-					(reference "C10")
-					(unit 1)
-				)
+					(reference "C9")
+					(unit 1)
+				)

Commit message: rough routing is complete (04.04.2025)
Parts:
- removed R2: 10k, Resistor_SMD:R_0603_1608Metric, symbol Device:R
- removed SW2: MSS-12D16, user:MSS-12D16, symbol Switch:SW_SPDT
Connections:
- net MPL_TEMP_1_3V3: now also U1.58 (PB6)
- net MPL_TEMP_2_3V3: now also U1.57 (PB5)
- net MPL_TEMP_0_3V3: now reaches U1.59 (PB7)

Commit message: 18.04.2025_final
Connections:
- net SPI1_CS_2: now also U1.15 (PA1)
Changed lines of the file:
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@@
 	(global_label "SPI1_CS_2"
 		(shape input)
-		(at 82.55 35.56 0)
+		(at 78.74 35.56 0)
 		(fields_autoplaced yes)
 		(effects
@@
 		)
 		(property "Intersheetrefs" "${INTERSHEET_REFS}"
-			(at 95.4532 35.56 0)
+			(at 91.6432 35.56 0)
 			(effects
 				(font

Commit message: 19.04.2025
Parts:
- added R2: 10k, Resistor_SMD:R_0603_1608Metric, symbol Device:R
Connections:
- net BOOT0: now also R2.2
- net GND: now also R2.1
