File: KiCad/BMS/power.kicad_sch (KiCad schematic)
At the start: 14 parts, among them U3 ST1S14PHR, U4 LDL1117S33R

Commit message: 22.03.2025
Other:
- note removed: "3V3 POWER LDO"
- moved on the sheet: C16, C17, C18, C19, C20, C21, C22, D2, L2, R4, R5, R6

Commit message: 23.03.2025
Other:
- note added: "ПОСЧИТАТЬ КОНДЕНСАТОР И РЕЗИСТРЫ"
Changed lines of the file:
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@@
+		)
+	)
+	(text "ПОСЧИТАТЬ КОНДЕНСАТОР И РЕЗИСТРЫ"
+		(exclude_from_sim no)
+		(at 99.06 71.12 0)
+		(effects
+			(font
+				(size 1.27 1.27)
+			)
 		)
 	)

Commit message: 25.03.2025
Parts:
- C22: renamed from C17; footprint Capacitor_THT:CP_Radial_D5.0mm_P2.00mm -> Capacitor_THT:CP_Radial_D6.3mm_P2.50mm; Ссылка https://www.promelec.ru/product/323633/ -> https://www.chipdip.ru/product0/14560
- renumbered C20 to C17, C21 to C18, C18 to C19, C19 to C20, C22 to C21
Changed lines of the file:
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@@
 		(on_board yes)
 		(dnp no)
-		(property "Reference" "C18"
+		(property "Reference" "C19"
 			(at 66.04 100.33 0)
 			(effects
@@
 			(project "BMS"
 				(path "/d2402062-308b-4eb4-ada9-28eaf3edc216/1af78963-9fe3-4dd0-8f03-a203e27f1081"
-					(reference "C18")
+					(reference "C19")
 					(unit 1)
 				)
@@
 		(on_board yes)
 		(dnp no)
-		(property "Reference" "C22"
+		(property "Reference" "C21"
 			(at 132.08 101.6 90)
 			(effects
@@
 			(project "BMS"
 				(path "/d2402062-308b-4eb4-ada9-28eaf3edc216/1af78963-9fe3-4dd0-8f03-a203e27f1081"
-					(reference "C22")
+					(reference "C21")
 					(unit 1)
 				)
@@
 		(dnp no)
 		(fields_autoplaced yes)
-		(property "Reference" "C17"
+		(property "Reference" "C22"
 			(at 137.16 108.6738 0)
 			(effects
@@
 			)
 		)
-		(property "Footprint" "Capacitor_THT:CP_Radial_D5.0mm_P2.00mm"
+		(property "Footprint" "Capacitor_THT:CP_Radial_D6.3mm_P2.50mm"
 			(at 134.62 110.49 0)
 			(effects
@@
 			)
 		)
-		(property "Ссылка" "https://www.promelec.ru/product/323633/"
+		(property "Ссылка" "https://www.chipdip.ru/product0/14560"
 			(at 134.62 110.49 0)
 			(effects
@@
 			(project "BMS"
 				(path "/d2402062-308b-4eb4-ada9-28eaf3edc216/1af78963-9fe3-4dd0-8f03-a203e27f1081"
-					(reference "C17")
+					(reference "C22")
 					(unit 1)
 				)
@@
 		(on_board yes)
 		(dnp no)
-		(property "Reference" "C20"
+		(property "Reference" "C17"
 			(at 201.93 101.6001 0)
 			(effects
@@
 			(project "BMS"
 				(path "/d2402062-308b-4eb4-ada9-28eaf3edc216/1af78963-9fe3-4dd0-8f03-a203e27f1081"
-					(reference "C20")
+					(reference "C17")
 					(unit 1)
 				)
@@
 		(on_board yes)
 		(dnp no)
-		(property "Reference" "C21"
+		(property "Reference" "C18"
 			(at 241.3 101.6001 0)
 			(effects
@@
 			(project "BMS"
 				(path "/d2402062-308b-4eb4-ada9-28eaf3edc216/1af78963-9fe3-4dd0-8f03-a203e27f1081"
-					(reference "C21")
+					(reference "C18")
 					(unit 1)
 				)
@@
 		(on_board yes)
 		(dnp no)
-		(property "Reference" "C19"
+		(property "Reference" "C20"
 			(at 73.66 100.33 0)
 			(effects
@@
 			(project "BMS"
 				(path "/d2402062-308b-4eb4-ada9-28eaf3edc216/1af78963-9fe3-4dd0-8f03-a203e27f1081"
-					(reference "C19")
-					(unit 1)
-				)
+					(reference "C20")
+					(unit 1)
+				)

Commit message: 30.03.2025
Parts:
- added J8: 430450400, Connector_Molex:Molex_Micro-Fit_3.0_43045-0400_2x02_P3.00mm_Horizontal, symbol Connector_Generic:Conn_02x02_Counter_Clockwise
Connections:
- net 24V0: now also J8.1 (Pin_1), J8.2 (Pin_2)
- net GND: now also J8.3 (Pin_3), J8.4 (Pin_4)

Commit message: rough routing is complete (04.04.2025)
Parts:
- renumbered C16 to C18, C17 to C19, C18 to C20, C19 to C21, C20 to C22, C21 to C23, C22 to C24, J8 to J5, U3 to U4, U4 to U5
Changed lines of the file:
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@@
 		(on_board yes)
 		(dnp no)
-		(property "Reference" "C19"
+		(property "Reference" "C21"
 			(at 66.04 100.33 0)
 			(effects
@@
 			(project "BMS"
 				(path "/d2402062-308b-4eb4-ada9-28eaf3edc216/1af78963-9fe3-4dd0-8f03-a203e27f1081"
-					(reference "C19")
+					(reference "C21")
 					(unit 1)
 				)
@@
 		(dnp no)
 		(fields_autoplaced yes)
-		(property "Reference" "U3"
+		(property "Reference" "U4"
 			(at 92.71 81.28 0)
 			(effects
@@
 			(project ""
 				(path "/d2402062-308b-4eb4-ada9-28eaf3edc216/1af78963-9fe3-4dd0-8f03-a203e27f1081"
-					(reference "U3")
+					(reference "U4")
 					(unit 1)
 				)
@@
 		(on_board yes)
 		(dnp no)
-		(property "Reference" "C21"
+		(property "Reference" "C23"
 			(at 132.08 101.6 90)
 			(effects
@@
 			(project "BMS"
 				(path "/d2402062-308b-4eb4-ada9-28eaf3edc216/1af78963-9fe3-4dd0-8f03-a203e27f1081"
-					(reference "C21")
+					(reference "C23")
 					(unit 1)
 				)
@@
 		(dnp no)
 		(fields_autoplaced yes)
-		(property "Reference" "C22"
+		(property "Reference" "C24"
 			(at 137.16 108.6738 0)
 			(effects
@@
 			(project "BMS"
 				(path "/d2402062-308b-4eb4-ada9-28eaf3edc216/1af78963-9fe3-4dd0-8f03-a203e27f1081"
-					(reference "C22")
+					(reference "C24")
 					(unit 1)
 				)
@@
 		(dnp no)
 		(fields_autoplaced yes)
-		(property "Reference" "#PWR068"
+		(property "Reference" "#PWR031"
 			(at 199.39 50.8 0)
 			(effects
@@
 			(project "BMS"
 				(path "/d2402062-308b-4eb4-ada9-28eaf3edc216/1af78963-9fe3-4dd0-8f03-a203e27f1081"
-					(reference "#PWR068")
+					(reference "#PWR031")
 					(unit 1)
 				)
@@
 		(on_board yes)
 		(dnp no)
-		(property "Reference" "#PWR067"
+		(property "Reference" "#PWR030"
 			(at 181.61 38.1 0)
 			(effects
@@
 			(project "BMS"
 				(path "/d2402062-308b-4eb4-ada9-28eaf3edc216/1af78963-9fe3-4dd0-8f03-a203e27f1081"
-					(reference "#PWR067")
+					(reference "#PWR030")
 					(unit 1)
 				)
@@
 		(on_board yes)
 		(dnp no)
-		(property "Reference" "#PWR022"
+		(property "Reference" "#PWR032"
 			(at 64.77 88.9 0)
 			(effects
@@
 			(project "BMS"
 				(path "/d2402062-308b-4eb4-ada9-28eaf3edc216/1af78963-9fe3-4dd0-8f03-a203e27f1081"
-					(reference "#PWR022")
+					(reference "#PWR032")
 					(unit 1)
 				)
@@
 		(on_board yes)
 		(dnp no)
-		(property "Reference" "C16"
+		(property "Reference" "C18"
 			(at 109.2199 85.09 0)
 			(effects
@@
 			(project "BMS"
 				(path "/d2402062-308b-4eb4-ada9-28eaf3edc216/1af78963-9fe3-4dd0-8f03-a203e27f1081"
-					(reference "C16")
+					(reference "C18")
 					(unit 1)
 				)
@@
 		(on_board yes)
 		(dnp no)
-		(property "Reference" "C17"
+		(property "Reference" "C19"
 			(at 201.93 101.6001 0)
 			(effects
@@
 			(project "BMS"
 				(path "/d2402062-308b-4eb4-ada9-28eaf3edc216/1af78963-9fe3-4dd0-8f03-a203e27f1081"
-					(reference "C17")
+					(reference "C19")
 					(unit 1)
 				)
@@
 		(on_board yes)
 		(dnp no)
-		(property "Reference" "C18"
+		(property "Reference" "C20"
 			(at 241.3 101.6001 0)
 			(effects
@@
 			(project "BMS"
 				(path "/d2402062-308b-4eb4-ada9-28eaf3edc216/1af78963-9fe3-4dd0-8f03-a203e27f1081"
-					(reference "C18")
+					(reference "C20")
 					(unit 1)
 				)
@@
 		(dnp no)
 		(fields_autoplaced yes)
-		(property "Reference" "J8"
+		(property "Reference" "J5"
 			(at 190.5 31.75 0)
 			(effects
@@
 			(project "BMS"
 				(path "/d2402062-308b-4eb4-ada9-28eaf3edc216/1af78963-9fe3-4dd0-8f03-a203e27f1081"
-					(reference "J8")
+					(reference "J5")
 					(unit 1)
 				)
@@
 		(on_board yes)
 		(dnp no)
-		(property "Reference" "C20"
+		(property "Reference" "C22"
 			(at 73.66 100.33 0)
 			(effects
@@
 			(project "BMS"
 				(path "/d2402062-308b-4eb4-ada9-28eaf3edc216/1af78963-9fe3-4dd0-8f03-a203e27f1081"
-					(reference "C20")
+					(reference "C22")
 					(unit 1)
 				)
@@
 		(dnp no)
 		(fields_autoplaced yes)
-		(property "Reference" "#PWR026"
+		(property "Reference" "#PWR036"
 			(at 205.74 121.92 0)
 			(effects
@@
 			(project "BMS"
 				(path "/d2402062-308b-4eb4-ada9-28eaf3edc216/1af78963-9fe3-4dd0-8f03-a203e27f1081"
-					(reference "#PWR026")
+					(reference "#PWR036")
 					(unit 1)
 				)
@@
 		(on_board yes)
 		(dnp no)
-		(property "Reference" "#PWR024"
+		(property "Reference" "#PWR034"
 			(at 205.74 88.9 0)
 			(effects
@@
 			(project "BMS"
 				(path "/d2402062-308b-4eb4-ada9-28eaf3edc216/1af78963-9fe3-4dd0-8f03-a203e27f1081"
-					(reference "#PWR024")
+					(reference "#PWR034")
 					(unit 1)
 				)
@@
 		(dnp no)
 		(fields_autoplaced yes)
-		(property "Reference" "#PWR027"
+		(property "Reference" "#PWR037"
 			(at 64.77 127 0)
 			(effects
@@
 			(project "BMS"
 				(path "/d2402062-308b-4eb4-ada9-28eaf3edc216/1af78963-9fe3-4dd0-8f03-a203e27f1081"
-					(reference "#PWR027")
+					(reference "#PWR037")
 					(unit 1)
 				)
@@
 		(on_board yes)
 		(dnp no)
-		(property "Reference" "U4"
+		(property "Reference" "U5"
 			(at 226.822 102.362 0)
 			(effects
@@
 			(project ""
 				(path "/d2402062-308b-4eb4-ada9-28eaf3edc216/1af78963-9fe3-4dd0-8f03-a203e27f1081"
-					(reference "U4")
+					(reference "U5")
 					(unit 1)
 				)
@@
 		(dnp no)
 		(fields_autoplaced yes)
-		(property "Reference" "#PWR025"
+		(property "Reference" "#PWR035"
 			(at 237.49 88.9 0)
 			(effects
@@
 			(project "BMS"
 				(path "/d2402062-308b-4eb4-ada9-28eaf3edc216/1af78963-9fe3-4dd0-8f03-a203e27f1081"
-					(reference "#PWR025")
+					(reference "#PWR035")
 					(unit 1)
 				)
@@
 		(on_board yes)
 		(dnp no)
-		(property "Reference" "#PWR023"
+		(property "Reference" "#PWR033"
 			(at 134.62 88.9 0)
 			(effects
@@
 			(project "BMS"
 				(path "/d2402062-308b-4eb4-ada9-28eaf3edc216/1af78963-9fe3-4dd0-8f03-a203e27f1081"
-					(reference "#PWR023")
-					(unit 1)
-				)
+					(reference "#PWR033")
+					(unit 1)
+				)

Commit message: 08.04.2025
Parts:
- renumbered R4 to R3, R5 to R4, R6 to R5
Connections:
- net 3V3: now also C19.2, U5.2 (V_OUT); no longer C20.2, U5.3 (V_IN)
- net 5V0: now also C20.2, U5.3 (V_IN); no longer C19.2, U5.2 (V_OUT)

Commit message: 19.04.2025
Parts:
- added R6: 220, Resistor_SMD:R_0603_1608Metric, symbol Device:R
- C21: renamed from C23; value C -> 150p
- L2: value 8u5 -> 6.8
- R4: renamed from R3; value 47k -> 10k
- R7: renamed from R5; value 2k7 -> 3k
- renumbered C21 to C19, C22 to C20, C19 to C22, C20 to C23, R4 to R5
Connections:
- net at C21.1, R4.1, U4.4 (FB): now also R6.2; no longer R7.2
- new net: R6.1, R7.2
Other:
- moved on the sheet: C18, C19, C20, C21, D2, L2, R4, R5, R7, U4

Commit message: 20.04.2025_true
Parts:
- L2: footprint user:CTSFW7050F -> user:CDCSAB0420-6R8M
Changed lines of the file:
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@@
 		(dnp no)
 		(property "Reference" "C21"
-			(at 132.715 83.82 90)
+			(at 125.73 93.345 90)
 			(effects
 				(font
@@
 			)
 		)
-		(property "Footprint" "user:CTSFW7050F"
+		(property "Footprint" "user:CDCSAB0420-6R8M"
 			(at 127 84.455 0)
 			(effects
@@
 			)
 		)
-		(property "Datasheet" "https://www.lcsc.com/datasheet/lcsc_datasheet_2311150110_Central-Semicon-CTSFW7050F-6R5M_C17401473.pdf"
+		(property "Datasheet" "https://www.chipdip.ru/product/csab0420-6r8m-6.8"
 			(at 127 84.455 0)
 			(effects
