File: KiCad/BMS/power.kicad_sch (KiCad schematic)
At the start: 16 parts, among them J5 430450400, U4 ST1S14PHR, U5 LDL1117S33R

Commit message: 21.04.2025_beta
Parts:
- L2: value 6.8 -> 6.8u
Changed lines of the file:
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@@
 		(fields_autoplaced yes)
 		(property "Reference" "L2"
-			(at 127 79.375 90)
+			(at 127 78.74 90)
 			(effects
 				(font
@@
 			)
 		)
-		(property "Value" "6.8"
-			(at 127 81.915 90)
+		(property "Value" "6.8u"
+			(at 127 81.28 90)
 			(effects
 				(font
